Commit message: fixed incorrect mesh paths

File: training/ref/demo_manipulation/robot_config/urdf/ur5_model.urdf.xacro (robot description, xacro)
@@ -4,5 +4,7 @@
        xmlns:interface="http://playerstage.sourceforge.net/gazebo/xmlschema/#interface"
        xmlns:xacro="http://ros.org/wiki/xacro">
-<include filename="$(find ur5_description)/urdf/arm.transmission.xacro" />
+  <include filename="$(find ur_description)/urdf/ur5.transmission.xacro" />
+  <include filename="$(find ur_description)/urdf/ur5.gazebo.xacro" />
+  <include filename="$(find ur_description)/urdf/materials.urdf.xacro" />
 <!--
 DH for UR5:
@@ -44,18 +46,18 @@
   <property name="forearm_radius" value="0.040" />    <!-- manually measured -->
   <property name="wrist_radius" value="0.045" />      <!-- manually measured -->
-<!-- Collision model -->
-  <property name="base_collision_length" value="0.160" />      <!-- manually measured -->
-  <property name="shoulder_collision_length" value="0.200" />  <!-- manually measured -->
-  <property name="shoulder_collision_offset" value="0.035" />  <!-- manually measured -->
-  <property name="elbow_collision_length" value="0.200" />     <!-- manually measured -->
-  <property name="elbow_collision_offset" value="0.035" />     <!-- manually measured -->
 <xacro:macro name="ur5_robot" params="prefix">
   <link name="${prefix}base_link" >
     <visual>
       <geometry>
-        <mesh filename="package://ur5_description/meshes/Base.dae" />
+		    <mesh filename="package://ur_description/meshes/ur5/visual/Base.dae" />
       </geometry>
       <origin xyz="0.0 0.0 0.003" rpy="0.0 0.0 ${3.0 * pi / 4.0}" />
     </visual>
+	<collision>
+      <geometry>
+        <mesh filename="package://ur_description/meshes/ur5/collision/Base.dae" />
+      </geometry>
+      <!-- <origin rpy="0.0 0.0 0.0" xyz="0.0 0.0 -0.009159"/> -->
+    </collision>
     <inertial>
       <mass value="${base_mass}" />
@@ -67,5 +69,5 @@
     <child link = "${prefix}shoulder_link" />
     <origin xyz="0.0 0.0 ${shoulder_height}" rpy="0.0 0.0 0.0" />
-    <axis xyz="0.0 0.0 1.0" />
+    <axis xyz="0 0 1" />
     <limit lower="${-0.75 * pi}" upper="${0.75 * pi}" effort="10.0" velocity="${pi}"/>
     <dynamics damping="10" friction="0.1"/>
@@ -74,12 +76,12 @@
     <visual>
       <geometry>
-        <mesh filename="package://ur5_description/meshes/Shoulder.dae" />
-      </geometry>
-    </visual>
-    <collision>
-      <geometry>
-        <cylinder length="${base_collision_length}" radius="${shoulder_radius}"/>
-      </geometry>
-      <origin xyz="0.0 0.0 ${-shoulder_height + (base_collision_length/2.0)}" rpy="0.0 0.0 0.0" />
+        <mesh filename="package://ur_description/meshes/ur5/visual/Shoulder.dae" />
+      </geometry>
+    </visual>
+    <collision>
+      <geometry>
+        <mesh filename="package://ur_description/meshes/ur5/collision/Shoulder.dae" />
+      </geometry>
+      <!-- <origin rpy="0.0 0.0 0.0" xyz="0.0 0.0 -0.009159"/> -->
     </collision>
     <inertial>
@@ -93,5 +95,5 @@
     <child link = "${prefix}upper_arm_link" />
     <origin xyz="0.0 ${shoulder_offset} 0.0" rpy="0.0 ${pi / 2.0} 0.0" />
-    <axis xyz="0.0 1.0 0.0" />
+    <axis xyz="0 1 0" />
     <limit lower="${-1.0 * pi}" upper="${1.0 * pi}" effort="10.0" velocity="${pi}"/>
     <dynamics damping="10" friction="0.1"/>
@@ -100,5 +102,5 @@
     <visual>
       <geometry>
-        <mesh filename="package://ur5_description/meshes/UpperArm.dae" />
+        <mesh filename="package://ur_description/meshes/ur5/visual/UpperArm.dae" />
       </geometry>
       <origin xyz="0.0 0.0 0.0" rpy="0.0 0.0 0.0" />
@@ -106,7 +108,7 @@
     <collision>
       <geometry>
-        <cylinder length="${upper_arm_length}" radius="${upper_arm_radius}"/>
-      </geometry>
-      <origin xyz="0.0 0.0 ${upper_arm_length/2.0}" rpy="0.0 0.0 0.0" />
+        <mesh filename="package://ur_description/meshes/ur5/collision/UpperArm.dae" />
+      </geometry>
+<!--       <origin rpy="0.0 0.0 0.0" xyz="0.0 0.0 0.2125"/> -->
     </collision>
     <inertial>
@@ -120,5 +122,5 @@
     <child link = "${prefix}forearm_link" />
     <origin xyz="0.0 ${-elbow_offset} ${upper_arm_length}" rpy="0.0 0.0 0.0" />
-    <axis xyz="0.0 1.0 0.0" />
+    <axis xyz="0 1 0" />
     <limit lower="${-0.2 * pi}" upper="${0.9 * pi}" effort="10.0" velocity="${pi}"/>
     <dynamics damping="10" friction="0.1"/>
@@ -127,12 +129,12 @@
     <visual>
       <geometry>
-        <mesh filename="package://ur5_description/meshes/Forearm.dae" />
-      </geometry>
-    </visual>
-    <collision>
-      <geometry>
-        <cylinder length="${forearm_length}" radius="${forearm_radius}"/>
-      </geometry>
-      <origin xyz="0.0 0.0 ${forearm_length/2.0}" rpy="0.0 0.0 0.0" />
+        <mesh filename="package://ur_description/meshes/ur5/visual/Forearm.dae" />
+      </geometry>
+    </visual>
+    <collision>
+      <geometry>
+        <mesh filename="package://ur_description/meshes/ur5/collision/Forearm.dae" />
+      </geometry>
+<!--       <origin rpy="0.0 0.0 0.0" xyz="0.0 0.0 0.196125"/> -->
     </collision>
     <inertial>
@@ -146,5 +148,5 @@
     <child link = "${prefix}wrist_1_link" />
     <origin xyz="0.0 0.0 ${forearm_length}" rpy="0.0 ${pi / 2.0} 0.0" />
-    <axis xyz="0.0 1.0 0.0" />
+    <axis xyz="0 1 0" />
     <limit lower="${-1.0 * pi}" upper="${0.01 * pi}" effort="10.0" velocity="${pi}"/>
     <dynamics damping="10" friction="0.1"/>
@@ -153,5 +155,5 @@
     <visual>
       <geometry>
-        <mesh filename="package://ur5_description/meshes/Wrist1.dae" />
+        <mesh filename="package://ur_description/meshes/ur5/visual/Wrist1.dae" />
       </geometry>
       <origin xyz="0.0 ${wrist_1_length} 0.0" rpy="0.0 ${pi / 2.0} 0.0" />
@@ -159,7 +161,7 @@
     <collision>
       <geometry>
-        <cylinder length="${1.6*wrist_1_length}" radius="${wrist_radius}"/>
-      </geometry>
-      <origin xyz="0.0 ${0.25*wrist_1_length} 0.0" rpy="${-pi/2.0} 0.0 0.0" />
+        <mesh filename="package://ur_description/meshes/ur5/collision/Wrist1.dae" />
+      </geometry>
+      <origin rpy="0.0 1.570796325 0.0" xyz="0.0 0.093 0.0"/>
     </collision>
     <inertial>
@@ -173,5 +175,5 @@
     <child link = "${prefix}wrist_2_link" />
     <origin xyz="0.0 ${wrist_1_length} 0.0" rpy="0.0 0.0 0.0" />
-    <axis xyz="0.0 0.0 1.0" />
+    <axis xyz="0 0 1" />
     <limit lower="${-1.0 * pi}" upper="${1.0 * pi}" effort="10.0" velocity="${pi}"/>
     <dynamics damping="10" friction="0.1"/>
@@ -180,5 +182,5 @@
     <visual>
       <geometry>
-        <mesh filename="package://ur5_description/meshes/Wrist2.dae" />
+        <mesh filename="package://ur_description/meshes/ur5/visual/Wrist2.dae" />
       </geometry>
       <origin xyz="0.0 0.0 ${wrist_2_length}" rpy="0.0 0.0 0.0" />
@@ -186,7 +188,7 @@
     <collision>
       <geometry>
-        <cylinder length="${1.6*wrist_2_length}" radius="${wrist_radius}"/>
-      </geometry>
-      <origin xyz="0.0 0.0 ${0.25*wrist_2_length}" rpy="0.0 0.0 0.0" />
+        <mesh filename="package://ur_description/meshes/ur5/collision/Wrist2.dae" />
+      </geometry>
+       <origin rpy="0.0 0.0 0.0" xyz="0.0 0.0 0.09465"/>
     </collision>
     <inertial>
@@ -200,5 +202,5 @@
     <child link = "${prefix}wrist_3_link" />
     <origin xyz="0.0 0.0 ${wrist_2_length}" rpy="0.0 0.0 0.0" />
-    <axis xyz="0.0 1.0 0.0" />
+    <axis xyz="0 1 0" />
     <limit lower="${-1.5 * pi}" upper="${1.5 * pi}" effort="10.0" velocity="${pi}"/>
     <dynamics damping="10" friction="0.1"/>
@@ -207,12 +209,11 @@
     <visual>
       <geometry>
-        <mesh filename="package://ur5_description/meshes/Wrist3.dae" />
-      </geometry>
-    </visual>
-    <collision>
-      <geometry>
-        <cylinder length="${1.65*wrist_3_length}" radius="${wrist_radius}"/>
-      </geometry>
-      <origin xyz="0.0 ${0.15 * wrist_3_length} 0.0" rpy="${-pi/2.0} 0.0 0.0" />
+        <mesh filename="package://ur_description/meshes/ur5/visual/Wrist3.dae" />
+      </geometry>
+    </visual>
+    <collision>
+      <geometry>
+        <mesh filename="package://ur_description/meshes/ur5/collision/Wrist3.dae" />
+      </geometry>
     </collision>
     <inertial>
@@ -228,31 +229,4 @@
   </joint>
   <link name="${prefix}ee_link" />
-  <!-- Extra links for collision model -->
-  <!-- Somehow don't work with gazebo TODO: fix this
-  <joint name="${prefix}shoulder_collision_joint" type="fixed">
-    <parent link="${prefix}upper_arm_link" />
-    <child link = "${prefix}shoulder_collision_link" />
-  </joint>
-  <link name="${prefix}shoulder_collision_link">
-    <collision>
-      <geometry>
-        <cylinder length="${shoulder_collision_length}" radius="${shoulder_radius}"/>
-      </geometry>
-      <origin xyz="0.0 ${-shoulder_collision_offset} 0.0" rpy="${-pi / 2.0} 0.0 0.0" />
-    </collision>
-  </link>
-  <joint name="${prefix}elbow_collision_joint" type="fixed">
-    <parent link="${prefix}upper_arm_link" />
-    <child link = "${prefix}elbow_collision_link" />
-  </joint>
-  <link name="${prefix}elbow_collision_link">
-    <collision>
-      <geometry>
-        <cylinder length="${elbow_collision_length}" radius="${elbow_radius}"/>
-      </geometry>
-      <origin xyz="0.0 ${-elbow_collision_offset} ${upper_arm_length}" rpy="${pi / 2.0} 0.0 0.0" />
-    </collision>
-  </link>
-  -->
   <xacro:ur_arm_transmission name="${prefix}" />
   <gazebo reference="universal_robot">

Commit message: added back wall and attached object link to arm.  substituted the 'include' keyword with 'xacro:include' since it is now deprecated in hydro

File: training/ref/demo_manipulation/robot_config/urdf/ur5_model.urdf.xacro (robot description, xacro)
@@ -4,7 +4,7 @@
        xmlns:interface="http://playerstage.sourceforge.net/gazebo/xmlschema/#interface"
        xmlns:xacro="http://ros.org/wiki/xacro">
-  <include filename="$(find ur_description)/urdf/ur5.transmission.xacro" />
-  <include filename="$(find ur_description)/urdf/ur5.gazebo.xacro" />
-  <include filename="$(find ur_description)/urdf/materials.urdf.xacro" />
+  <xacro:include filename="$(find ur_description)/urdf/ur5.transmission.xacro" />
+  <xacro:include filename="$(find ur_description)/urdf/ur5.gazebo.xacro" />
+  <xacro:include filename="$(find ur_description)/urdf/materials.urdf.xacro" />
 <!--
 DH for UR5:

File: training/ref/demo_manipulation/robot_config/urdf/ur5_workspace.urdf (robot description, URDF)
Before this commit: robot ur5_workspace, 29 links, 28 joints
Links:
- added link attached_object_link; collision box size=0.17 0.17 0.17
- added link back_wall2; collision box size=0.04 2.0 1; visual box size=0.04 2.0 1
Joints:
- added joint tcp_to_attached_object: type fixed, parent tcp_frame, child attached_object_link, origin xyz=0 0 0.085
- added joint world_frame_to_back_wall2: type fixed, parent world_frame, child back_wall2, origin xyz=0.2 0 0.5 rpy=0 0 0

File: training/ref/demo_manipulation/robot_config/urdf/ur5_workspace.xacro (robot description, xacro)
@@ -1,12 +1,15 @@
 <?xml version="1.0" ?>
 <robot name="ur5_workspace" xmlns:xacro="http://ros.org/wiki/xacro">
-	<include filename="$(find robot_config)/urdf/vacuum_gripper_macro.xacro"/>
-  	<include filename="$(find robot_config)/urdf/ur5_model.urdf.xacro" />
-	<include filename="$(find robot_config)/urdf/workspace_components.xacro"/>
-	<include filename="$(find robot_config)/urdf/kinect_sensor_macro.xacro"/>
+	<xacro:include filename="$(find robot_config)/urdf/vacuum_gripper_macro.xacro"/>
+  	<xacro:include filename="$(find robot_config)/urdf/ur5_model.urdf.xacro" />
+	<xacro:include filename="$(find robot_config)/urdf/workspace_components.xacro"/>
+	<xacro:include filename="$(find robot_config)/urdf/kinect_sensor_macro.xacro"/>
 	<!-- property list -->
 	<xacro:property name="workcell_height" value="1"/>
 	<xacro:property name="robot_stand_height" value="0.20"/>
 	<xacro:property name="vacuum_gripper_width" value="0.088"/>
+        <xacro:property name="attached_object_length" value="0.17"/>
+	<xacro:property name="attached_object_width" value="0.17"/>
+	<xacro:property name="attached_object_height" value="0.17"/>
 	<xacro:property name="arm_prefix" value=""/>
 	<!-- instantiating arm and gripper -->
@@ -47,4 +50,12 @@
 		</collision>
 	</link>
+	<link name="attached_object_link">
+		<collision>
+			<geometry>
+				<box size="${attached_object_length} ${attached_object_width} ${attached_object_height}"/>
+			</geometry>
+			<material name="blue_transparent"/>
+		</collision>
+	</link>
 	<!-- instantiating sensor definitions -->
 	<xacro:sensor_definitions prefix="${arm_prefix}" parent_link="ur5_stand"
@@ -66,4 +77,9 @@
 		<origin xyz="-0.238 0 ${robot_stand_height}"/>
 	</joint>
+	<joint name="tcp_to_attached_object" type="fixed">
+		<parent link="tcp_frame"/>
+		<child link="attached_object_link"/>
+		<origin xyz="0 0 ${0.5 * attached_object_height}"/>
+	</joint>
 	<!-- end of arm-workcell link definitions -->
 	<!-- arm-workcell joint definitions -->

File: training/ref/demo_manipulation/robot_config/urdf/workspace_components.xacro (robot description, xacro)
@@ -133,6 +133,6 @@
 		<xacro:workcell_element name="front_wall2" parent="world_frame"
 			 length="0.1" width="2.220" height="${workcell_height}" offset_x="-1.3375" offset_y="0"/>
-		<!--<xacro:workcell_element name="back_wall2" parent="world_frame"
-			 length="0.04" width="2.00" height="${workcell_height}" offset_x="0.20" offset_y="0"/>-->
+		<xacro:workcell_element name="back_wall2" parent="world_frame"
+			 length="0.04" width="2.00" height="${workcell_height}" offset_x="0.20" offset_y="0"/>
 		<xacro:workcell_element name="left_wall2" parent="world_frame"
 			length="1.384" width="0.1" height="${workcell_height}" offset_x="-0.601" offset_y="1.060"/>
