Commit message: changed the size of the gripper_body

File: training/ref/demo_manipulation/robot_config/urdf/vacuum_gripper_macro.xacro (robot description, xacro)
@@ -5,5 +5,5 @@
 	<xacro:property name="gripper_width" value="0.088"/>
 	<xacro:property name="gripper_height" value="0.0946"/>
-	<xacro:property name="gripper_body_height" value="0.14"/>-->
+	<xacro:property name="gripper_body_height" value="0.15"/>
 	<xacro:macro name="vacuum_gripper_definition" params="prefix gripper_adjustment">
 		<link name="${prefix}gripper_frame"/>
@@ -25,5 +25,5 @@
 				<!--<origin xyz="0 0 0.03"/>-->
 				<geometry>
-					<box size="${gripper_length} ${gripper_width} ${gripper_height}"/>
+					<box size="${gripper_length} ${gripper_width} ${gripper_body_height}"/>
 				</geometry>
 				<material name="another_blue2">
