Commit message: regenerated urdf from new xacro

File: training/ref/demo_manipulation/robot_config/urdf/ur5_workspace.urdf (robot description, URDF)
Before this commit: robot ur5_workspace, 26 links, 25 joints
Links:
- link base_link: geometry collision mesh filename=package://ur_description/meshes/ur5/collision/Base.dae; visual mesh filename=package://ur_description/meshes/ur5/visual/Base.dae
- link forearm_link: geometry collision mesh filename=package://ur_description/meshes/ur5/collision/Forearm.dae; visual mesh filename=package://ur_description/meshes/ur5/visual/Forearm.dae
- link shoulder_link: geometry collision mesh filename=package://ur_description/meshes/ur5/collision/Shoulder.dae; visual mesh filename=package://ur_description/meshes/ur5/visual/Shoulder.dae
- link upper_arm_link: geometry collision mesh filename=package://ur_description/meshes/ur5/collision/UpperArm.dae; visual mesh filename=package://ur_description/meshes/ur5/visual/UpperArm.dae
- link wrist_1_link: geometry collision mesh filename=package://ur_description/meshes/ur5/collision/Wrist1.dae; visual mesh filename=package://ur_description/meshes/ur5/visual/Wrist1.dae
- link wrist_2_link: geometry collision mesh filename=package://ur_description/meshes/ur5/collision/Wrist2.dae; visual mesh filename=package://ur_description/meshes/ur5/visual/Wrist2.dae
- link wrist_3_link: geometry collision mesh filename=package://ur_description/meshes/ur5/collision/Wrist3.dae; visual mesh filename=package://ur_description/meshes/ur5/visual/Wrist3.dae
Joints:
- joint elbow_joint: axis 0.0 1.0 0.0 -> 0 1 0
- joint shoulder_lift_joint: axis 0.0 1.0 0.0 -> 0 1 0
- joint shoulder_pan_joint: axis 0.0 0.0 1.0 -> 0 0 1
- joint wrist_1_joint: axis 0.0 1.0 0.0 -> 0 1 0
- joint wrist_2_joint: axis 0.0 0.0 1.0 -> 0 0 1
- joint wrist_3_joint: axis 0.0 1.0 0.0 -> 0 1 0

Commit message: added cylinder around base to eliminate unnecessary collision checks with the sensor data

File: training/ref/demo_manipulation/robot_config/urdf/ur5_workspace.urdf (robot description, URDF)
Before this commit: robot ur5_workspace, 26 links, 25 joints
Links:
- added link octomap_keepout; collision cylinder length=0.4 radius=0.14
Joints:
- added joint world_to_octomap_keepout: type fixed, parent world_frame, child octomap_keepout, origin xyz=-0.238 0 0.2

File: training/ref/demo_manipulation/robot_config/urdf/ur5_workspace.xacro (robot description, xacro)
@@ -31,4 +31,12 @@
 		</collision>
 	</link>
+	<link name="octomap_keepout">
+		<collision>
+			<geometry>
+				<cylinder radius="0.14" length="${robot_stand_height * 2}"/>
+			</geometry>
+			<material name="blue_transparent"/>
+		</collision>
+	</link>
 	<!-- instantiating sensor definitions -->
 	<xacro:sensor_definitions prefix="${arm_prefix}" parent_link="ur5_stand"
@@ -39,4 +47,9 @@
 		<child link="ur5_stand"/>
 		<origin xyz="-0.238 0 ${robot_stand_height * 0.5}"/>
+	</joint>
+	<joint name="world_to_octomap_keepout" type="fixed">
+		<parent link="world_frame"/>
+		<child link="octomap_keepout"/>
+		<origin xyz="-0.238 0 ${robot_stand_height}"/>
 	</joint>
 	<!-- end of arm-workcell link definitions -->

Commit message: added roof to the cell in order to bound the arm movements in the z direction

File: training/ref/demo_manipulation/robot_config/urdf/ur5_workspace.urdf (robot description, URDF)
Before this commit: robot ur5_workspace, 27 links, 26 joints
Links:
- added link roof2; collision box size=1.3875 2.22 0.04
Joints:
- added joint workcell_to_roof2: type fixed, parent world_frame, child roof2, origin xyz=-0.69375 0 0 rpy=0 0 0

File: training/ref/demo_manipulation/robot_config/urdf/workspace_components.xacro (robot description, xacro)
@@ -5,4 +5,5 @@
 	<xacro:property name="workcell_length" value="2.775"/>
 	<xacro:property name="workcell_width" value="2.220"/>
+	<xacro:property name="workcell_thickness" value="0.04"/>
 	<!-- color macros -->
 	<xacro:macro name="material_yellow_transparent">
@@ -111,7 +112,21 @@
 			</collision>
 		</link>
+		<link name="roof2">
+			<collision>
+				<origin xyz="0 0 ${workcell_height }" rpy="0 0 0"/>
+				<xacro:workcell_geometry length="${workcell_length * 0.5}"
+					 width="${workcell_width}" height="${workcell_thickness}">
+					<material name="blue_transparent"/>
+				</xacro:workcell_geometry>
+			</collision>
+		</link>
 		<joint name="workcell_to_table_base2" type="fixed">
 			<parent link="world_frame"/>
 			<child link="table_base2"/>
+			<origin xyz="${workcell_length * -0.25} 0 0" rpy="0 0 0"/>
+		</joint>
+		<joint name="workcell_to_roof2" type="fixed">
+			<parent link="world_frame"/>
+			<child link="roof2"/>
 			<origin xyz="${workcell_length * -0.25} 0 0" rpy="0 0 0"/>
 		</joint>

Commit message: changes to environment.  Need to clean up vacuum gripper xacro file

File: training/ref/demo_manipulation/robot_config/urdf/ur5_workspace.urdf (robot description, URDF)
Before this commit: robot ur5_workspace, 28 links, 27 joints
Links:
- removed link octomap_keepout
- added link base_padding; collision cylinder length=0.4 radius=0.14
- added link wrist_3_padding; collision cylinder length=0.12 radius=0.14
Joints:
- removed joint world_to_octomap_keepout
- added joint world_to_base_padding: type fixed, parent world_frame, child base_padding, origin xyz=-0.238 0 0.2
- added joint wrist_3_link_to_wrist_3_padding: type fixed, parent wrist_3_link, child wrist_3_padding, origin xyz=0 0.09 0 rpy=1.57 0 0

File: training/ref/demo_manipulation/robot_config/urdf/ur5_workspace.xacro (robot description, xacro)
@@ -31,8 +31,16 @@
 		</collision>
 	</link>
-	<link name="octomap_keepout">
+	<link name="base_padding">
 		<collision>
 			<geometry>
 				<cylinder radius="0.14" length="${robot_stand_height * 2}"/>
+			</geometry>
+			<material name="blue_transparent"/>
+		</collision>
+	</link>
+	<link name="wrist_3_padding">
+		<collision>
+			<geometry>
+				<cylinder radius="0.14" length="0.12"/>
 			</geometry>
 			<material name="blue_transparent"/>
@@ -48,7 +56,12 @@
 		<origin xyz="-0.238 0 ${robot_stand_height * 0.5}"/>
 	</joint>
-	<joint name="world_to_octomap_keepout" type="fixed">
+	<joint name="wrist_3_link_to_wrist_3_padding" type="fixed">
+		<parent link="wrist_3_link"/>
+		<child link="wrist_3_padding"/>
+		<origin xyz="0 0.09 0" rpy="1.57 0 0"/>
+	</joint>
+	<joint name="world_to_base_padding" type="fixed">
 		<parent link="world_frame"/>
-		<child link="octomap_keepout"/>
+		<child link="base_padding"/>
 		<origin xyz="-0.238 0 ${robot_stand_height}"/>
 	</joint>

File: training/ref/demo_manipulation/robot_config/urdf/vacuum_gripper_macro.xacro (robot description, xacro)
@@ -5,4 +5,5 @@
 	<xacro:property name="gripper_width" value="0.088"/>
 	<xacro:property name="gripper_height" value="0.0946"/>
+	<xacro:property name="gripper_body_height" value="0.14"/>-->
 	<xacro:macro name="vacuum_gripper_definition" params="prefix gripper_adjustment">
 		<link name="${prefix}gripper_frame"/>
@@ -22,4 +23,5 @@
 			</visual>
 			<collision>
+				<!--<origin xyz="0 0 0.03"/>-->
 				<geometry>
 					<box size="${gripper_length} ${gripper_width} ${gripper_height}"/>

Commit message: added back wall

File: training/ref/demo_manipulation/robot_config/urdf/ur5_workspace.urdf (robot description, URDF)
Before this commit: robot ur5_workspace, 29 links, 28 joints
Links:
- added link back_wall2; collision box size=0.04 2.0 1; visual box size=0.04 2.0 1
- link wrist_3_padding: geometry collision cylinder length=0.12 radius=0.10
Joints:
- added joint world_frame_to_back_wall2: type fixed, parent world_frame, child back_wall2, origin xyz=0.2 0 0.5 rpy=0 0 0

File: training/ref/demo_manipulation/robot_config/urdf/ur5_workspace.xacro (robot description, xacro)
@@ -42,5 +42,5 @@
 		<collision>
 			<geometry>
-				<cylinder radius="0.14" length="0.12"/>
+				<cylinder radius="0.10" length="0.12"/>
 			</geometry>
 			<material name="blue_transparent"/>

File: training/ref/demo_manipulation/robot_config/urdf/workspace_components.xacro (robot description, xacro)
@@ -133,6 +133,6 @@
 		<xacro:workcell_element name="front_wall2" parent="world_frame"
 			 length="0.1" width="2.220" height="${workcell_height}" offset_x="-1.3375" offset_y="0"/>
-		<!--xacro:workcell_element name="back_wall2" parent="world_frame"
-			 length="0.04" width="2.00" height="${workcell_height}" offset_x="-0.02" offset_y="0"/-->
+		<xacro:workcell_element name="back_wall2" parent="world_frame"
+			 length="0.04" width="2.00" height="${workcell_height}" offset_x="0.20" offset_y="0"/>
 		<xacro:workcell_element name="left_wall2" parent="world_frame"
 			length="1.384" width="0.1" height="${workcell_height}" offset_x="-0.601" offset_y="1.060"/>

Commit message: removed back_wall_2 object since it was causing issues with tf

File: training/ref/demo_manipulation/robot_config/urdf/ur5_workspace.urdf (robot description, URDF)
Before this commit: robot ur5_workspace, 30 links, 29 joints
Links:
- removed link back_wall2
Joints:
- removed joint world_frame_to_back_wall2

File: training/ref/demo_manipulation/robot_config/urdf/workspace_components.xacro (robot description, xacro)
@@ -133,6 +133,6 @@
 		<xacro:workcell_element name="front_wall2" parent="world_frame"
 			 length="0.1" width="2.220" height="${workcell_height}" offset_x="-1.3375" offset_y="0"/>
-		<xacro:workcell_element name="back_wall2" parent="world_frame"
-			 length="0.04" width="2.00" height="${workcell_height}" offset_x="0.20" offset_y="0"/>
+		<!--<xacro:workcell_element name="back_wall2" parent="world_frame"
+			 length="0.04" width="2.00" height="${workcell_height}" offset_x="0.20" offset_y="0"/>-->
 		<xacro:workcell_element name="left_wall2" parent="world_frame"
 			length="1.384" width="0.1" height="${workcell_height}" offset_x="-0.601" offset_y="1.060"/>
@@ -144,4 +144,4 @@
 			 length="0.121" width="0.260" height="0.14" offset_x="-0.012" offset_y="-0.465"/>
 	</xacro:macro>
-	<!-- end of workcell part1 components macro -->
+	<!-- end of workcell part2 components macro -->
 </robot>

Commit message: increased gripper collision model height

File: training/ref/demo_manipulation/robot_config/urdf/ur5_workspace.urdf (robot description, URDF)
Before this commit: robot ur5_workspace, 31 links, 30 joints
Links:
- link gripper_body: geometry collision box size=0.044 0.088 0.16; visual mesh filename=package://robot_config/meshes/vacuum_gripper_single_suction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

File: training/ref/demo_manipulation/robot_config/urdf/vacuum_gripper_macro.xacro (robot description, xacro)
@@ -5,5 +5,5 @@
 	<xacro:property name="gripper_width" value="0.088"/>
 	<xacro:property name="gripper_height" value="0.0946"/>
-	<xacro:property name="gripper_body_height" value="0.15"/>
+	<xacro:property name="gripper_body_height" value="0.16"/>
 	<xacro:macro name="vacuum_gripper_definition" params="prefix gripper_adjustment">
 		<link name="${prefix}gripper_frame"/>
