Commit message: removed attached object link from robot arm

File: training/ref/demo_manipulation/robot_config/urdf/ur5_collision_avoidance.urdf (robot description, URDF)
Before this commit: robot ur5_collision_avoidance, 31 links, 30 joints
Links:
- removed link attached_object_link
Joints:
- removed joint tcp_to_attached_object

File: training/ref/demo_manipulation/robot_config/urdf/ur5_collision_avoidance.xacro (robot description, xacro)
@@ -50,5 +50,5 @@
 		</collision>
 	</link>
-	<link name="attached_object_link">
+	<!--<link name="attached_object_link">
 		<collision>
 			<geometry>
@@ -57,5 +57,5 @@
 			<material name="blue_transparent"/>
 		</collision>
-	</link>
+	</link>-->
 	<!-- instantiating sensor definitions -->
 	<xacro:sensor_definitions prefix="${arm_prefix}" parent_link="ur5_stand"
@@ -77,9 +77,9 @@
 		<origin xyz="-0.238 0 ${robot_stand_height}"/>
 	</joint>
-	<joint name="tcp_to_attached_object" type="fixed">
+	<!--<joint name="tcp_to_attached_object" type="fixed">
 		<parent link="tcp_frame"/>
 		<child link="attached_object_link"/>
 		<origin xyz="0 0 ${0.5 * attached_object_height}"/>
-	</joint>
+	</joint>-->
 	<!-- end of arm-workcell link definitions -->
 	<!-- arm-workcell joint definitions -->

Commit message: re-enabled attached_box_link

File: training/ref/demo_manipulation/robot_config/urdf/ur5_collision_avoidance.urdf (robot description, URDF)
Before this commit: robot ur5_collision_avoidance, 30 links, 29 joints
Links:
- added link attached_object_link; collision box size=0.17 0.17 0.17
Joints:
- added joint tcp_to_attached_object: type fixed, parent tcp_frame, child attached_object_link, origin xyz=0 0 0.085

File: training/ref/demo_manipulation/robot_config/urdf/ur5_collision_avoidance.xacro (robot description, xacro)
@@ -50,5 +50,5 @@
 		</collision>
 	</link>
-	<!--<link name="attached_object_link">
+	<link name="attached_object_link">
 		<collision>
 			<geometry>
@@ -57,5 +57,5 @@
 			<material name="blue_transparent"/>
 		</collision>
-	</link>-->
+	</link>
 	<!-- instantiating sensor definitions -->
 	<xacro:sensor_definitions prefix="${arm_prefix}" parent_link="ur5_stand"
@@ -77,9 +77,9 @@
 		<origin xyz="-0.238 0 ${robot_stand_height}"/>
 	</joint>
-	<!--<joint name="tcp_to_attached_object" type="fixed">
+	<joint name="tcp_to_attached_object" type="fixed">
 		<parent link="tcp_frame"/>
 		<child link="attached_object_link"/>
 		<origin xyz="0 0 ${0.5 * attached_object_height}"/>
-	</joint>-->
+	</joint>
 	<!-- end of arm-workcell link definitions -->
 	<!-- arm-workcell joint definitions -->

Commit message: added small geometry to tcp_frame link in  ur5_collision_avoidance.xacro file and updated moveit config package.  Copied changes from groovy to read the touch links parameter and use then during motion path planning

File: training/ref/demo_manipulation/robot_config/urdf/ur5_collision_avoidance.urdf (robot description, URDF)
Before this commit: robot ur5_collision_avoidance, 30 links, 29 joints
Links:
- link tcp_frame: geometry collision sphere radius=0.005; visual sphere radius=0.005

File: training/ref/demo_manipulation/robot_config/urdf/ur5_workspace.urdf (robot description, URDF)
Before this commit: robot ur5_workspace, 26 links, 25 joints
Links:
- added link back_wall2; collision box size=0.04 2.0 1; visual box size=0.04 2.0 1
- added link roof2; collision box size=1.3875 2.22 0.04
- link gripper_body: geometry collision box size=0.044 0.088 0.16; visual mesh filename=package://robot_config/meshes/vacuum_gripper_single_suction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
- link tcp_frame: geometry collision sphere radius=0.005; visual sphere radius=0.005
Joints:
- added joint workcell_to_roof2: type fixed, parent world_frame, child roof2, origin xyz=-0.69375 0 0 rpy=0 0 0
- added joint world_frame_to_back_wall2: type fixed, parent world_frame, child back_wall2, origin xyz=0.2 0 0.5 rpy=0 0 0

File: training/ref/demo_manipulation/robot_config/urdf/ur5_workspace.xacro (robot description, xacro)
@@ -1,8 +1,8 @@
 <?xml version="1.0" ?>
 <robot name="ur5_workspace" xmlns:xacro="http://ros.org/wiki/xacro">
-	<include filename="$(find robot_config)/urdf/vacuum_gripper_macro.xacro"/>
-  	<include filename="$(find robot_config)/urdf/ur5_model.urdf.xacro" />
-	<include filename="$(find robot_config)/urdf/workspace_components.xacro"/>
-	<include filename="$(find robot_config)/urdf/kinect_sensor_macro.xacro"/>
+	<xacro:include filename="$(find robot_config)/urdf/vacuum_gripper_macro.xacro"/>
+  	<xacro:include filename="$(find robot_config)/urdf/ur5_model.urdf.xacro" />
+	<xacro:include filename="$(find robot_config)/urdf/workspace_components.xacro"/>
+	<xacro:include filename="$(find robot_config)/urdf/kinect_sensor_macro.xacro"/>
 	<!-- property list -->
 	<xacro:property name="workcell_height" value="1"/>

File: training/ref/demo_manipulation/robot_config/urdf/vacuum_gripper_macro.xacro (robot description, xacro)
@@ -32,5 +32,19 @@
 			</collision>
 		</link>
-		<link name="${prefix}tcp_frame"/>
+		<link name="${prefix}tcp_frame">
+			<visual>
+				<geometry>
+					<sphere radius="0.005"/>
+				</geometry>
+				<material name="white">
+					<color rgba="1 1 1 0.5"/>
+				</material>
+			</visual>
+			<collision>
+				<geometry>
+					<sphere radius="0.005"/>
+				</geometry>
+			</collision>
+		</link>
 		<joint name="${prefix}gripper_to_palm" type="fixed">
 			<parent link="${prefix}gripper_frame"/>
