Commit message: replaced universal_robot metapackage with new code which supports the io interface

File: training/supplements/src/universal_robot/ur_description/urdf/ur10.urdf.xacro (robot description, xacro)
@@ -4,7 +4,7 @@
        xmlns:interface="http://playerstage.sourceforge.net/gazebo/xmlschema/#interface"
        xmlns:xacro="http://ros.org/wiki/xacro">
-  <include filename="$(find ur_description)/urdf/ur10.transmission.xacro" />
-  <include filename="$(find ur_description)/urdf/ur10.gazebo.xacro" />
-  <include filename="$(find ur_description)/urdf/materials.urdf.xacro" />
+  <xacro:include filename="$(find ur_description)/urdf/ur10.transmission.xacro" />
+  <xacro:include filename="$(find ur_description)/urdf/ur10.gazebo.xacro" />
+  <xacro:include filename="$(find ur_description)/urdf/materials.urdf.xacro" />
   <property name="pi" value="3.14159265" />
   <!-- Inertia parameters -->
@@ -67,6 +67,6 @@
 		<origin xyz="0.0 0.0 ${shoulder_height}" rpy="0.0 0.0 0.0" />
 		<axis xyz="0.0 0.0 1.0" />
-		<limit lower="${-2.0 * pi}" upper="${2.0 * pi}" effort="10.0" velocity="${pi}"/>
-		<dynamics damping="10" friction="0.1"/>
+		<limit lower="${-2.0 * pi}" upper="${2.0 * pi}" effort="330.0" velocity="2.16"/>
+		<dynamics damping="1.2" friction="0.0"/>
 	</joint>
 	<link name="${prefix}shoulder_link">
@@ -94,5 +94,5 @@
 		<axis xyz="0.0 1.0 0.0" />
 		<limit lower="${-2.0 * pi}" upper="${2.0 * pi}" effort="10.0" velocity="${pi}"/>
-		<dynamics damping="10" friction="0.1"/>
+		<dynamics damping="1.2" friction="0.0"/>
 	</joint>
 	<link name="${prefix}upper_arm_link">
@@ -121,6 +121,6 @@
 		<origin xyz="0.0 ${-elbow_offset} ${upper_arm_length}" rpy="0.0 0.0 0.0" />
 		<axis xyz="0.0 1.0 0.0" />
-		<limit lower="${-2.0 * pi}" upper="${2.0 * pi}" effort="10.0" velocity="${pi}"/>
-		<dynamics damping="10" friction="0.1"/>
+		<limit lower="${-2.0 * pi}" upper="${2.0 * pi}" effort="150.0" velocity="${pi}"/>
+		<dynamics damping="0.6" friction="0.0"/>
 	</joint>
 	<link name="${prefix}forearm_link">
@@ -147,6 +147,6 @@
 		<origin xyz="0.0 0.0 ${forearm_length}" rpy="0.0 ${pi / 2.0} 0.0" />
 		<axis xyz="0.0 1.0 0.0" />
-		<limit lower="${-2.0 * pi}" upper="${2.0 * pi}" effort="10.0" velocity="${pi}"/>
-		<dynamics damping="10" friction="0.1"/>
+		<limit lower="${-2.0 * pi}" upper="${2.0 * pi}" effort="54.0" velocity="${pi}"/>
+		<dynamics damping="0.6" friction="0.0"/>
 	</joint>
 	<link name="${prefix}wrist_1_link">
@@ -175,6 +175,6 @@
 		<origin xyz="0.0 ${wrist_1_length} 0.0" rpy="0.0 0.0 0.0" />
 		<axis xyz="0.0 0.0 1.0" />
-		<limit lower="${-2.0 * pi}" upper="${2.0 * pi}" effort="10.0" velocity="${pi}"/>
-		<dynamics damping="10" friction="0.1"/>
+		<limit lower="${-2.0 * pi}" upper="${2.0 * pi}" effort="54.0" velocity="${pi}"/>
+		<dynamics damping="0.6" friction="0.0"/>
 	</joint>
 	<link name="${prefix}wrist_2_link">
@@ -203,6 +203,6 @@
 		<origin xyz="0.0 0.0 ${wrist_2_length}" rpy="0.0 0.0 0.0" />
 		<axis xyz="0.0 1.0 0.0" />
-		<limit lower="${-2.0 * pi}" upper="${2.0 * pi}" effort="10.0" velocity="${pi}"/>
-		<dynamics damping="10" friction="0.1"/>
+		<limit lower="${-2.0 * pi}" upper="${2.0 * pi}" effort="54.0" velocity="${pi}"/>
+		<dynamics damping="0.6" friction="0.0"/>
 	</joint>
 	<link name="${prefix}wrist_3_link">
@@ -226,6 +226,6 @@
 		</inertial>
 	</link>
-  <xacro:ur10_arm_transmission name="${prefix}" />
-  <xacro:ur10_arm_gazebo name="${prefix}" />
+  <xacro:ur10_arm_transmission prefix="${prefix}" />
+  <xacro:ur10_arm_gazebo prefix="${prefix}" />
   </xacro:macro>
 </robot>

File: training/supplements/src/universal_robot/ur_description/urdf/ur5.urdf.xacro (robot description, xacro)
@@ -4,7 +4,7 @@
        xmlns:interface="http://playerstage.sourceforge.net/gazebo/xmlschema/#interface"
        xmlns:xacro="http://ros.org/wiki/xacro">
-  <include filename="$(find ur_description)/urdf/ur5.transmission.xacro" />
-  <include filename="$(find ur_description)/urdf/ur5.gazebo.xacro" />
-  <include filename="$(find ur_description)/urdf/materials.urdf.xacro" />
+  <xacro:include filename="$(find ur_description)/urdf/ur5.transmission.xacro" />
+  <xacro:include filename="$(find ur_description)/urdf/ur5.gazebo.xacro" />
+  <xacro:include filename="$(find ur_description)/urdf/materials.urdf.xacro" />
 <!--
 DH for UR5:
@@ -70,6 +70,6 @@
     <origin xyz="0.0 0.0 ${shoulder_height}" rpy="0.0 0.0 0.0" />
     <axis xyz="0 0 1" />
-    <limit lower="${-2.0 * pi}" upper="${2.0 * pi}" effort="10.0" velocity="${pi}"/>
-    <dynamics damping="10" friction="0.1"/>
+    <limit lower="${-2.0 * pi}" upper="${2.0 * pi}" effort="150.0" velocity="${pi}"/>
+    <dynamics damping="0.4" friction="0.0"/>
   </joint>
   <link name="${prefix}shoulder_link">
@@ -96,6 +96,6 @@
     <origin xyz="0.0 ${shoulder_offset} 0.0" rpy="0.0 ${pi / 2.0} 0.0" />
     <axis xyz="0 1 0" />
-    <limit lower="${-2.0 * pi}" upper="${2.0 * pi}" effort="10.0" velocity="${pi}"/>
-    <dynamics damping="10" friction="0.1"/>
+    <limit lower="${-2.0 * pi}" upper="${2.0 * pi}" effort="150.0" velocity="${pi}"/>
+    <dynamics damping="0.4" friction="0.0"/>
   </joint>
   <link name="${prefix}upper_arm_link">
@@ -123,6 +123,6 @@
     <origin xyz="0.0 ${-elbow_offset} ${upper_arm_length}" rpy="0.0 0.0 0.0" />
     <axis xyz="0 1 0" />
-    <limit lower="${-2.0 * pi}" upper="${2.0 * pi}" effort="10.0" velocity="${pi}"/>
-    <dynamics damping="10" friction="0.1"/>
+    <limit lower="${-2.0 * pi}" upper="${2.0 * pi}" effort="150.0" velocity="${pi}"/>
+    <dynamics damping="0.4" friction="0.0"/>
   </joint>
   <link name="${prefix}forearm_link">
@@ -149,6 +149,6 @@
     <origin xyz="0.0 0.0 ${forearm_length}" rpy="0.0 ${pi / 2.0} 0.0" />
     <axis xyz="0 1 0" />
-    <limit lower="${-1.0 * pi}" upper="${0.25 * pi}" effort="10.0" velocity="${pi}"/>
-    <dynamics damping="10" friction="0.1"/>
+    <limit lower="${-1.0 * pi}" upper="${0.25 * pi}" effort="28.0" velocity="${pi}"/>
+    <dynamics damping="0.3" friction="0.0"/>
   </joint>
   <link name="${prefix}wrist_1_link">
@@ -176,6 +176,6 @@
     <origin xyz="0.0 ${wrist_1_length} 0.0" rpy="0.0 0.0 0.0" />
     <axis xyz="0 0 1" />
-    <limit lower="${-1.0 * pi}" upper="${1.0 * pi}" effort="10.0" velocity="${pi}"/>
-    <dynamics damping="10" friction="0.1"/>
+    <limit lower="${-1.0 * pi}" upper="${1.0 * pi}" effort="28.0" velocity="${pi}"/>
+    <dynamics damping="0.3" friction="0.0"/>
   </joint>
   <link name="${prefix}wrist_2_link">
@@ -203,6 +203,6 @@
     <origin xyz="0.0 0.0 ${wrist_2_length}" rpy="0.0 0.0 0.0" />
     <axis xyz="0 1 0" />
-    <limit lower="${-1.0 * pi}" upper="${1.0 * pi}" effort="10.0" velocity="${pi}"/>
-    <dynamics damping="10" friction="0.1"/>
+    <limit lower="${-1.0 * pi}" upper="${1.0 * pi}" effort="28.0" velocity="${pi}"/>
+    <dynamics damping="0.3" friction="0.0"/>
   </joint>
   <link name="${prefix}wrist_3_link">
@@ -229,5 +229,5 @@
   </joint>
   <link name="${prefix}ee_link" />
-  <xacro:ur_arm_transmission name="${prefix}" />
+  <xacro:ur5_arm_transmission name="${prefix}" />
   <gazebo reference="universal_robot">
     <material>Gazebo/Blue</material>
