Commit message: Fixed empty tool rotation so that parts placed correctly

File: training/work/2.5/src/lesson_advanced_launch/models/empty_tool.xacro (robot description, xacro)
@@ -13,5 +13,5 @@
     <parent link="tool_base" />
     <child link="tool1" />
-    <origin xyz="0 0 0" rpy="0 0 ${0*deg}" />
+    <origin xyz="0 0 0" rpy="0 0 ${-90*deg}" />
   </joint>
   <!-- tool1 is the point that parts connect to the tool -->
