Commit message: intial demo_motoman_manipulation in indigo

File: training/supplements/src/motoman_config/cfg/sia20d_mesh_macro.xacro (robot description, xacro)
@@ -133,5 +133,4 @@
 			</collision>
 		</link>
-		<link name="${prefix}tool0" />
 		<!-- end of link list -->
 		<!-- joint list -->
@@ -185,9 +184,4 @@
 			<limit lower="-3.1416" upper="3.1416" effort="100" velocity="6.97" />
 		</joint>
-		<joint name="${prefix}link_t-tool0" type="fixed" >
-            <origin xyz="0 0 0.0" rpy="0 -1.571 0"/>
-            <parent link="${prefix}link_t" />
-            <child link="${prefix}tool0" />
-        </joint>
 		<!-- end of joint list -->
 	</xacro:macro>
