Commit message: Simplify Exercise 2.4 (remove extra options)

File: training/orig/2.4/src/lesson_tf/models/environment.xacro (robot description, xacro)
@@ -1,5 +1,4 @@
 <?xml version="1.0"?>
-<robot xmlns:xacro="http://ros.org/wiki/xacro" name="ses_environment">
-  <include filename="$(find xacro_properties)/properties.xacro" /> <!--contains properties such as "pi" and "deg"-->
+<robot xmlns:xacro="http://ros.org/wiki/xacro" name="environment">
   <!-- link "world" and connected joints -->
   <link name="world" />
@@ -7,10 +6,10 @@
     <parent link="world" />
     <child link="base_link" />
-    <origin xyz="0 0 0" rpy="0 ${0*deg} 0" />
+    <origin xyz="0 0 0" rpy="0 0 0" />
   </joint>
   <joint name="world-grinder" type="fixed" >
     <parent link="world" />
     <child link="grinder" />
-    <origin xyz="0.523 -0.609 0.6226" rpy="${-90*deg} 0 ${45*deg}" />
+    <origin xyz="0.523 -0.609 0.6226" rpy="${-90*3.14159/180} 0 ${45*3.14159/180}" />
   </joint>
   <!-- link "grinder" and connected joints -->
@@ -18,10 +17,10 @@
     <visual>
       <geometry>
-        <mesh filename="package://lesson_tf_terminal/models/grinder_visual.dae" />
+        <mesh filename="package://lesson_tf/models/grinder_visual.dae" />
       </geometry>
     </visual>
     <collision>
       <geometry>
-        <mesh filename="package://lesson_tf_terminal/models/grinder_collision.dae" />
+        <mesh filename="package://lesson_tf/models/grinder_collision.dae" />
       </geometry>
     </collision>
