Commit message: update 3.7 for indigo

File: training/orig/3.7/src/workcell_config/urdf/workcell.urdf (robot description, URDF)
Before this commit: robot workcell, 15 links, 14 joints
Links:
- added link base
- link base_link: geometry collision mesh filename=package://abb_irb2400_support/meshes/irb2400/collision/base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; visual mesh filename=package://abb_irb2400_support/meshes/irb2400/visual/base_li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
- link link_1: geometry collision mesh filename=package://abb_irb2400_support/meshes/irb2400/collision/link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; visual mesh filename=package://abb_irb2400_support/meshes/irb2400/visual/link_1.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
- link link_2: geometry collision mesh filename=package://abb_irb2400_support/meshes/irb2400/collision/link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; visual mesh filename=package://abb_irb2400_support/meshes/irb2400/visual/link_2.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
- link link_3: geometry collision mesh filename=package://abb_irb2400_support/meshes/irb2400/collision/link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; visual mesh filename=package://abb_irb2400_support/meshes/irb2400/visual/link_3.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
- link link_4: geometry collision mesh filename=package://abb_irb2400_support/meshes/irb2400/collision/link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; visual mesh filename=package://abb_irb2400_support/meshes/irb2400/visual/link_4.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
- link link_5: geometry collision mesh filename=package://abb_irb2400_support/meshes/irb2400/collision/link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; visual mesh filename=package://abb_irb2400_support/meshes/irb2400/visual/link_5.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
- link link_6: geometry collision mesh filename=package://abb_irb2400_support/meshes/irb2400/collision/link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; visual mesh filename=package://abb_irb2400_support/meshes/irb2400/visual/link_6.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
Joints:
- added joint base_link-base: type fixed, parent base_link, child base, origin xyz=0 0 0 rpy=0 0 0
- joint joint_6-tool0: origin xyz=0 0 0 rpy=0 0 0 -> xyz=0 0 0 rpy=0 1.57079632679 0

File: training/orig/3.7/src/workcell_config/urdf/workcell.xacro (robot description, xacro)
@@ -2,7 +2,7 @@
 <robot name="workcell" xmlns:xacro="http://ros.org/wiki/xacro">
 	<xacro:include filename="$(find workcell_config)/urdf/table.xacro"/>
-  <xacro:include filename="$(find abb_common)/urdf/irb_2400_macro.xacro"/>
+  <xacro:include filename="$(find abb_irb2400_support)/urdf/irb2400_macro.xacro"/>
   <link name="world_frame"/>
-  <xacro:irb_2400 prefix=""/>
+  <xacro:abb_irb2400 prefix=""/>
   <joint name="world_to_robot" type="fixed">
     <parent link="world_frame"/>
