Commit message: update demo_ur5: further constrain, update launch to prevent conflicting robot_descriptions

File: training/orig/demo_ur5/src/workcell_config/urdf/workcell.xacro (robot description, xacro)
@@ -39,5 +39,5 @@
     <parent link="world" />
     <child link="left_wall" />
-    <origin xyz="0.0 -1.0 0.0" rpy="0.0 0.0 0.0" />
+    <origin xyz="0.0 -0.5 0.0" rpy="0.0 0.0 0.0" />
   </joint>
   <link name="right_wall">
@@ -52,5 +52,5 @@
     <parent link="world" />
     <child link="right_wall" />
-    <origin xyz="0.0 1.0 0.0" rpy="0.0 0.0 0.0" />
+    <origin xyz="0.0 0.5 0.0" rpy="0.0 0.0 0.0" />
   </joint>
   <link name="back_wall">
@@ -65,5 +65,5 @@
     <parent link="world" />
     <child link="back_wall" />
-    <origin xyz="-0.5 0.0 0.0" rpy="0.0 0.0 0.0" />
+    <origin xyz="-0.3 0.0 0.0" rpy="0.0 0.0 0.0" />
   </joint>
 <!--  <link name="ceiling">
