Commit message: Revamped 1.8 and 2.1 with URDF/Xacro excercise.

File: training/ref/1.8/src/myworkcell_support/urdf/workcell.urdf (robot description, URDF)
Before this commit: robot table, 2 links, 1 joints
Links:
- removed link table_base
- added link world
Joints:
- joint base_to_table: origin (none) -> xyz=0 0 0.5 rpy=0 0 0; parent table_base -> world

File: training/ref/2.1/src/myworkcell_support/urdf/myworkcell.xacro (robot description, xacro)
@@ -1,3 +1,3 @@
-<?xml version="1.0" ?>
+<?xml version="1.0" encoding="UTF-8"?>
 <robot name="myworkcell" xmlns:xacro="http://ros.org/wiki/xacro">
   <xacro:include filename="$(find ur_description)/urdf/ur5.urdf.xacro"/>

Commit message: Added a 'camera_frame' link the URDF

File: training/ref/1.8/src/myworkcell_support/urdf/workcell.urdf (robot description, URDF)
Before this commit: robot workcell, 2 links, 1 joints
Links:
- added link camera_frame
Joints:
- removed joint base_to_table
- added joint world_to_camera: type fixed, parent world, child camera_frame, origin xyz=0 0 1.0 rpy=0 1.571 0
- added joint world_to_table: type fixed, parent world, child table, origin xyz=0 0 0.5 rpy=0 0 0

File: training/ref/2.1/src/myworkcell_support/urdf/workcell.xacro (robot description, xacro)
@@ -30,3 +30,9 @@
     <origin xyz="0 0 0" rpy="0 0 0"/>
   </joint>
+  <link name="camera_frame"/>
+  <joint name="world_to_camera" type="fixed">
+    <parent link="world"/>
+    <child link="camera_frame"/>
+    <origin xyz="0 0 1.0" rpy="0 1.571 0" />
+  </joint>
 </robot>

File: training/ref/2.3/src/myworkcell_support/urdf/workcell.xacro (robot description, xacro)
@@ -30,3 +30,9 @@
     <origin xyz="0 0 0" rpy="0 0 0"/>
   </joint>
+  <link name="camera_frame"/>
+  <joint name="world_to_camera" type="fixed">
+    <parent link="world"/>
+    <child link="camera_frame"/>
+    <origin xyz="0 0 1.0" rpy="0 1.571 0" />
+  </joint>
 </robot>

File: training/ref/2.4/src/myworkcell_support/urdf/workcell.xacro (robot description, xacro)
@@ -30,3 +30,9 @@
     <origin xyz="0 0 0" rpy="0 0 0"/>
   </joint>
+  <link name="camera_frame"/>
+  <joint name="world_to_camera" type="fixed">
+    <parent link="world"/>
+    <child link="camera_frame"/>
+    <origin xyz="0 0 1.0" rpy="0 1.571 0" />
+  </joint>
 </robot>

File: training/ref/2.5/src/myworkcell_support/urdf/workcell.xacro (robot description, xacro)
@@ -30,3 +30,9 @@
     <origin xyz="0 0 0" rpy="0 0 0"/>
   </joint>
+  <link name="camera_frame"/>
+  <joint name="world_to_camera" type="fixed">
+    <parent link="world"/>
+    <child link="camera_frame"/>
+    <origin xyz="0 0 1.0" rpy="0 1.571 0" />
+  </joint>
 </robot>
