Commit message: Fixed errors when launching demo caused by new version of ur_description

File: exercises/Descartes_Planning_and_Execution/src/ur5_demo_support/urdf/ur5.urdf.xacro (robot description, xacro)
@@ -1,6 +1,6 @@
 <?xml version="1.0"?>
 <robot xmlns:xacro="http://www.ros.org/wiki/xacro">
-  <xacro:include filename="$(find ur_description)/urdf/ur5.transmission.xacro" />
-  <xacro:include filename="$(find ur_description)/urdf/ur5.gazebo.xacro" />
+  <xacro:include filename="$(find ur_description)/urdf/ur.transmission.xacro" />
+  <xacro:include filename="$(find ur_description)/urdf/ur.gazebo.xacro" />
   <property name="pi" value="3.14159265" />
   <!-- Inertia parameters -->
@@ -72,5 +72,5 @@
       <visual>
         <geometry>
-          <mesh filename="package://ur_description/meshes/ur5/visual/Base.dae" />
+          <mesh filename="package://ur_description/meshes/ur5/visual/base.dae" />
         </geometry>
         <material name="LightGrey">
@@ -103,5 +103,5 @@
       <visual>
         <geometry>
-          <mesh filename="package://ur_description/meshes/ur5/visual/Shoulder.dae" />
+          <mesh filename="package://ur_description/meshes/ur5/visual/shoulder.dae" />
         </geometry>
         <material name="LightGrey">
@@ -134,13 +134,13 @@
       <visual>
         <geometry>
-          <mesh filename="package://ur_description/meshes/ur5/visual/UpperArm.dae" />
-        </geometry>
-        <material name="LightGrey">
-          <color rgba="0.7 0.7 0.7 1.0"/>
-        </material>
-      </visual>
-      <collision>
-        <geometry>
-          <mesh filename="package://ur_description/meshes/ur5/collision/upper_arm.stl" />
+          <mesh filename="package://ur_description/meshes/ur5/visual/upperarm.dae" />
+        </geometry>
+        <material name="LightGrey">
+          <color rgba="0.7 0.7 0.7 1.0"/>
+        </material>
+      </visual>
+      <collision>
+        <geometry>
+          <mesh filename="package://ur_description/meshes/ur5/collision/upperarm.stl" />
         </geometry>
       </collision>
@@ -165,5 +165,5 @@
       <visual>
         <geometry>
-          <mesh filename="package://ur_description/meshes/ur5/visual/Forearm.dae" />
+          <mesh filename="package://ur_description/meshes/ur5/visual/forearm.dae" />
         </geometry>
         <material name="LightGrey">
@@ -196,13 +196,13 @@
       <visual>
         <geometry>
-          <mesh filename="package://ur_description/meshes/ur5/visual/Wrist1.dae" />
-        </geometry>
-        <material name="LightGrey">
-          <color rgba="0.7 0.7 0.7 1.0"/>
-        </material>
-      </visual>
-      <collision>
-        <geometry>
-          <mesh filename="package://ur_description/meshes/ur5/collision/wrist_1.stl" />
+          <mesh filename="package://ur_description/meshes/ur5/visual/wrist1.dae" />
+        </geometry>
+        <material name="LightGrey">
+          <color rgba="0.7 0.7 0.7 1.0"/>
+        </material>
+      </visual>
+      <collision>
+        <geometry>
+          <mesh filename="package://ur_description/meshes/ur5/collision/wrist1.stl" />
         </geometry>
       </collision>
@@ -227,13 +227,13 @@
       <visual>
         <geometry>
-          <mesh filename="package://ur_description/meshes/ur5/visual/Wrist2.dae" />
-        </geometry>
-        <material name="LightGrey">
-          <color rgba="0.7 0.7 0.7 1.0"/>
-        </material>
-      </visual>
-      <collision>
-        <geometry>
-          <mesh filename="package://ur_description/meshes/ur5/collision/wrist_2.stl" />
+          <mesh filename="package://ur_description/meshes/ur5/visual/wrist2.dae" />
+        </geometry>
+        <material name="LightGrey">
+          <color rgba="0.7 0.7 0.7 1.0"/>
+        </material>
+      </visual>
+      <collision>
+        <geometry>
+          <mesh filename="package://ur_description/meshes/ur5/collision/wrist2.stl" />
         </geometry>
       </collision>
@@ -258,13 +258,13 @@
       <visual>
         <geometry>
-          <mesh filename="package://ur_description/meshes/ur5/visual/Wrist3.dae" />
-        </geometry>
-        <material name="LightGrey">
-          <color rgba="0.7 0.7 0.7 1.0"/>
-        </material>
-      </visual>
-      <collision>
-        <geometry>
-          <mesh filename="package://ur_description/meshes/ur5/collision/wrist_3.stl" />
+          <mesh filename="package://ur_description/meshes/ur5/visual/wrist3.dae" />
+        </geometry>
+        <material name="LightGrey">
+          <color rgba="0.7 0.7 0.7 1.0"/>
+        </material>
+      </visual>
+      <collision>
+        <geometry>
+          <mesh filename="package://ur_description/meshes/ur5/collision/wrist3.stl" />
         </geometry>
       </collision>
@@ -286,6 +286,6 @@
       </collision>
     </link>
-    <xacro:ur5_arm_transmission prefix="${prefix}" />
-    <xacro:ur5_arm_gazebo prefix="${prefix}" />
+    <xacro:ur_arm_transmission prefix="${prefix}" />
+    <xacro:ur_arm_gazebo prefix="${prefix}" />
   </xacro:macro>
 </robot>
