Commit message: Update Exercise 3.0 to match wiki

File: exercises/3.0/src/myworkcell_support/urdf/workcell.urdf (robot description, URDF)
Before this commit: robot workcell, 3 links, 2 joints
Links:
- link table: geometry collision box size=0.6 0.6 0.05; visual box size=0.6 0.6 0.05

Commit message: Minor tweaks to workcell URDF
- shift camera, to place target closer to robot
- adjust table size, to match latest wiki instructions

File: exercises/3.0/src/myworkcell_support/urdf/workcell.urdf (robot description, URDF)
Before this commit: robot myworkcell, 3 links, 2 joints
Links:
- link table: geometry collision box size=1.0 1.0 0.05; visual box size=1.0 1.0 0.05
Joints:
- joint world_to_camera: origin xyz=0 0 1.0 rpy=0 1.571 0 -> xyz=-0.25 -0.5 1.25 rpy=0 3.14159 0

File: exercises/3.1/src/myworkcell_support/urdf/workcell.xacro (robot description, xacro)
@@ -6,10 +6,10 @@
     <visual>
       <geometry>
-        <box size="0.6 0.6 0.05"/>
+        <box size="1.0 1.0 0.05"/>
       </geometry>
     </visual>
     <collision>
       <geometry>
-        <box size="0.6 0.6 0.05"/>
+        <box size="1.0 1.0 0.05"/>
       </geometry>
     </collision>
@@ -25,5 +25,5 @@
     <parent link="world"/>
     <child link="camera_frame"/>
-    <origin xyz="0 0 1.0" rpy="0 1.571 0"/>
+    <origin xyz="-0.25 -0.5 1.25" rpy="0 3.14159 0"/>
   </joint>
   <joint name="table_to_robot" type="fixed">

File: exercises/4.0/src/myworkcell_support/urdf/workcell.xacro (robot description, xacro)
@@ -6,10 +6,10 @@
     <visual>
       <geometry>
-        <box size="0.6 0.6 0.05"/>
+        <box size="1.0 1.0 0.05"/>
       </geometry>
     </visual>
     <collision>
       <geometry>
-        <box size="0.6 0.6 0.05"/>
+        <box size="1.0 1.0 0.05"/>
       </geometry>
     </collision>
@@ -25,5 +25,5 @@
     <parent link="world"/>
     <child link="camera_frame"/>
-    <origin xyz="0.5 0 1.0" rpy="0 3.14159 0"/>
+    <origin xyz="-0.25 -0.5 1.25" rpy="0 3.14159 0"/>
   </joint>
   <joint name="table_to_robot" type="fixed">

Commit message: Revert "Minor tweaks to workcell URDF"
This reverts commit 40bef29f3d4ff3e63ea17e0159b6edf19c3c39c0.

File: exercises/3.0/src/myworkcell_support/urdf/workcell.urdf (robot description, URDF)
Before this commit: robot myworkcell, 3 links, 2 joints
Links:
- link table: geometry collision box size=0.6 0.6 0.05; visual box size=0.6 0.6 0.05
Joints:
- joint world_to_camera: origin xyz=-0.25 -0.5 1.25 rpy=0 3.14159 0 -> xyz=0 0 1.0 rpy=0 1.571 0

File: exercises/3.1/src/myworkcell_support/urdf/workcell.xacro (robot description, xacro)
@@ -6,10 +6,10 @@
     <visual>
       <geometry>
-        <box size="1.0 1.0 0.05"/>
+        <box size="0.6 0.6 0.05"/>
       </geometry>
     </visual>
     <collision>
       <geometry>
-        <box size="1.0 1.0 0.05"/>
+        <box size="0.6 0.6 0.05"/>
       </geometry>
     </collision>
@@ -25,5 +25,5 @@
     <parent link="world"/>
     <child link="camera_frame"/>
-    <origin xyz="-0.25 -0.5 1.25" rpy="0 3.14159 0"/>
+    <origin xyz="0 0 1.0" rpy="0 1.571 0"/>
   </joint>
   <joint name="table_to_robot" type="fixed">

File: exercises/4.0/src/myworkcell_support/urdf/workcell.xacro (robot description, xacro)
@@ -6,10 +6,10 @@
     <visual>
       <geometry>
-        <box size="1.0 1.0 0.05"/>
+        <box size="0.6 0.6 0.05"/>
       </geometry>
     </visual>
     <collision>
       <geometry>
-        <box size="1.0 1.0 0.05"/>
+        <box size="0.6 0.6 0.05"/>
       </geometry>
     </collision>
@@ -25,5 +25,5 @@
     <parent link="world"/>
     <child link="camera_frame"/>
-    <origin xyz="-0.25 -0.5 1.25" rpy="0 3.14159 0"/>
+    <origin xyz="0.5 0 1.0" rpy="0 3.14159 0"/>
   </joint>
   <joint name="table_to_robot" type="fixed">
