Commit message: Added edited files that were corrected

File: exercises/4.0/src/myworkcell_support/urdf/workcell.xacro (robot description, xacro)
@@ -2,4 +2,5 @@
 <robot name="myworkcell" xmlns:xacro="http://ros.org/wiki/xacro">
   <xacro:include filename="$(find ur_description)/urdf/ur5.urdf.xacro" />
+<xacro:ur5_robot prefix="" joint_limited="true"/>
   <link name="world"/>
   <link name="table">
@@ -16,5 +17,4 @@
   </link>
   <link name="camera_frame"/>
-  <xacro:ur5_robot prefix="" joint_limited="true"/>
   <joint name="world_to_table" type="fixed">
     <parent link="world"/>
@@ -25,5 +25,5 @@
     <parent link="world"/>
     <child link="camera_frame"/>
-    <origin xyz="0 0 1.0" rpy="0 1.571 0"/>
+    <origin xyz="0.5 0 1.0" rpy="0 3.14159 0"/>
   </joint>
   <joint name="table_to_robot" type="fixed">

File: exercises/4.1/src/myworkcell_support/urdf/workcell.xacro (robot description, xacro)
@@ -25,5 +25,5 @@
     <parent link="world"/>
     <child link="camera_frame"/>
-    <origin xyz="0 0 1.0" rpy="0 3.14159 0"/>
+    <origin xyz="0.5 0 1.0" rpy="0 3.14159 0"/>
   </joint>
   <joint name="table_to_robot" type="fixed">

Commit message: Revert "Added edited files that were corrected"
This reverts commit 51b08993ccf45bd874eaef56e0bb456c7ba73fc7.

File: exercises/4.0/src/myworkcell_support/urdf/workcell.xacro (robot description, xacro)
@@ -2,5 +2,4 @@
 <robot name="myworkcell" xmlns:xacro="http://ros.org/wiki/xacro">
   <xacro:include filename="$(find ur_description)/urdf/ur5.urdf.xacro" />
-<xacro:ur5_robot prefix="" joint_limited="true"/>
   <link name="world"/>
   <link name="table">
@@ -17,4 +16,5 @@
   </link>
   <link name="camera_frame"/>
+  <xacro:ur5_robot prefix="" joint_limited="true"/>
   <joint name="world_to_table" type="fixed">
     <parent link="world"/>
@@ -25,5 +25,5 @@
     <parent link="world"/>
     <child link="camera_frame"/>
-    <origin xyz="0.5 0 1.0" rpy="0 3.14159 0"/>
+    <origin xyz="0 0 1.0" rpy="0 1.571 0"/>
   </joint>
   <joint name="table_to_robot" type="fixed">

File: exercises/4.1/src/myworkcell_support/urdf/workcell.xacro (robot description, xacro)
@@ -25,5 +25,5 @@
     <parent link="world"/>
     <child link="camera_frame"/>
-    <origin xyz="0.5 0 1.0" rpy="0 3.14159 0"/>
+    <origin xyz="0 0 1.0" rpy="0 3.14159 0"/>
   </joint>
   <joint name="table_to_robot" type="fixed">
