Commit message: perception demo now works with latest universal robot repo

File: exercises/Perception-Driven_Manipulation/solution_ws/src/robot_config/urdf/ur5.urdf.xacro (robot description, xacro)
@@ -1,6 +1,6 @@
 <?xml version="1.0"?>
-<robot xmlns:xacro="http://www.ros.org/wiki/xacro">
-  <xacro:include filename="$(find ur_description)/urdf/ur5.transmission.xacro" />
-  <xacro:include filename="$(find ur_description)/urdf/ur5.gazebo.xacro" />
+<robot xmlns:xacro="http://ros.org/wiki/xacro">
+  <xacro:include filename="$(find ur_description)/urdf/ur.transmission.xacro" />
+  <xacro:include filename="$(find ur_description)/urdf/ur.gazebo.xacro" />
   <!-- Inertia parameters -->
   <property name="base_mass" value="4.0" />  <!-- This mass might be incorrect -->
@@ -71,5 +71,5 @@
       <visual>
         <geometry>
-          <mesh filename="package://ur_description/meshes/ur5/visual/Base.dae" />
+          <mesh filename="package://ur_description/meshes/ur5/visual/base.dae" />
         </geometry>
         <material name="LightGrey">
@@ -102,5 +102,5 @@
       <visual>
         <geometry>
-          <mesh filename="package://ur_description/meshes/ur5/visual/Shoulder.dae" />
+          <mesh filename="package://ur_description/meshes/ur5/visual/shoulder.dae" />
         </geometry>
         <material name="LightGrey">
@@ -133,13 +133,13 @@
       <visual>
         <geometry>
-          <mesh filename="package://ur_description/meshes/ur5/visual/UpperArm.dae" />
-        </geometry>
-        <material name="LightGrey">
-          <color rgba="0.7 0.7 0.7 1.0"/>
-        </material>
-      </visual>
-      <collision>
-        <geometry>
-          <mesh filename="package://ur_description/meshes/ur5/collision/upper_arm.stl" />
+          <mesh filename="package://ur_description/meshes/ur5/visual/upperarm.dae" />
+        </geometry>
+        <material name="LightGrey">
+          <color rgba="0.7 0.7 0.7 1.0"/>
+        </material>
+      </visual>
+      <collision>
+        <geometry>
+          <mesh filename="package://ur_description/meshes/ur5/collision/upperarm.stl" />
         </geometry>
       </collision>
@@ -164,5 +164,5 @@
       <visual>
         <geometry>
-          <mesh filename="package://ur_description/meshes/ur5/visual/Forearm.dae" />
+          <mesh filename="package://ur_description/meshes/ur5/visual/forearm.dae" />
         </geometry>
         <material name="LightGrey">
@@ -195,13 +195,13 @@
       <visual>
         <geometry>
-          <mesh filename="package://ur_description/meshes/ur5/visual/Wrist1.dae" />
-        </geometry>
-        <material name="LightGrey">
-          <color rgba="0.7 0.7 0.7 1.0"/>
-        </material>
-      </visual>
-      <collision>
-        <geometry>
-          <mesh filename="package://ur_description/meshes/ur5/collision/wrist_1.stl" />
+          <mesh filename="package://ur_description/meshes/ur5/visual/wrist1.dae" />
+        </geometry>
+        <material name="LightGrey">
+          <color rgba="0.7 0.7 0.7 1.0"/>
+        </material>
+      </visual>
+      <collision>
+        <geometry>
+          <mesh filename="package://ur_description/meshes/ur5/collision/wrist1.stl" />
         </geometry>
       </collision>
@@ -226,13 +226,13 @@
       <visual>
         <geometry>
-          <mesh filename="package://ur_description/meshes/ur5/visual/Wrist2.dae" />
-        </geometry>
-        <material name="LightGrey">
-          <color rgba="0.7 0.7 0.7 1.0"/>
-        </material>
-      </visual>
-      <collision>
-        <geometry>
-          <mesh filename="package://ur_description/meshes/ur5/collision/wrist_2.stl" />
+          <mesh filename="package://ur_description/meshes/ur5/visual/wrist2.dae" />
+        </geometry>
+        <material name="LightGrey">
+          <color rgba="0.7 0.7 0.7 1.0"/>
+        </material>
+      </visual>
+      <collision>
+        <geometry>
+          <mesh filename="package://ur_description/meshes/ur5/collision/wrist2.stl" />
         </geometry>
       </collision>
@@ -257,13 +257,13 @@
       <visual>
         <geometry>
-          <mesh filename="package://ur_description/meshes/ur5/visual/Wrist3.dae" />
-        </geometry>
-        <material name="LightGrey">
-          <color rgba="0.7 0.7 0.7 1.0"/>
-        </material>
-      </visual>
-      <collision>
-        <geometry>
-          <mesh filename="package://ur_description/meshes/ur5/collision/wrist_3.stl" />
+          <mesh filename="package://ur_description/meshes/ur5/visual/wrist3.dae" />
+        </geometry>
+        <material name="LightGrey">
+          <color rgba="0.7 0.7 0.7 1.0"/>
+        </material>
+      </visual>
+      <collision>
+        <geometry>
+          <mesh filename="package://ur_description/meshes/ur5/collision/wrist3.stl" />
         </geometry>
       </collision>
@@ -285,6 +285,6 @@
       </collision>
     </link>
-    <xacro:ur5_arm_transmission prefix="${prefix}" />
-    <xacro:ur5_arm_gazebo prefix="${prefix}" />
+    <xacro:ur_arm_transmission prefix="${prefix}" />
+    <xacro:ur_arm_gazebo prefix="${prefix}" />
   </xacro:macro>
 </robot>

File: exercises/Perception-Driven_Manipulation/solution_ws/src/robot_config/urdf/ur5_collision_avoidance.xacro (robot description, xacro)
@@ -1,73 +1,73 @@
 <?xml version="1.0" ?>
 <robot name="ur5_collision_avoidance" xmlns:xacro="http://ros.org/wiki/xacro">
-	<xacro:include filename="$(find robot_config)/urdf/vacuum_gripper_macro.xacro"/>
-  <xacro:include filename="$(find robot_config)/urdf/ur5.urdf.xacro" />
-	<xacro:include filename="$(find robot_config)/urdf/workspace_components.xacro"/>
-	<xacro:include filename="$(find robot_config)/urdf/kinect_sensor_macro.xacro"/>
-	<!-- property list -->
-	<xacro:property name="workcell_height" value="1"/>
-	<xacro:property name="robot_stand_height" value="0.20"/>
-	<xacro:property name="vacuum_gripper_width" value="0.088"/>
-        <xacro:property name="attached_object_length" value="0.17"/>
-	<xacro:property name="attached_object_width" value="0.17"/>
-	<xacro:property name="attached_object_height" value="0.17"/>
-	<xacro:property name="arm_prefix" value=""/>
-	<!-- instantiating arm and gripper -->
-  <xacro:ur5_robot prefix="" joint_limited="true"/>
-	<xacro:vacuum_gripper_definition prefix="${arm_prefix}" gripper_adjustment="0.01"/>
-	<!-- instantiating workcell definitions -->
-	<xacro:workcell_zone2_components/>
-	<!-- end of workcell definitions -->
-	<!-- arm-workcell link definitions -->
-	<link name="ur5_stand">
-		<visual>
-			<geometry>
-				<cylinder radius="0.0735" length="${robot_stand_height}"/>
-			</geometry>
-			<material name="orange_transparent"/>
-		</visual>
-		<collision>
-			<geometry>
-				<cylinder radius="0.0735" length="${robot_stand_height}"/>
-			</geometry>
-			<material name="blue_transparent"/>
-		</collision>
-	</link>
-	<link name="base_padding">
-		<collision>
-			<geometry>
-				<cylinder radius="0.14" length="${robot_stand_height * 2}"/>
-			</geometry>
-			<material name="blue_transparent"/>
-		</collision>
-	</link>
-	<!-- instantiating sensor definitions -->
-        <xacro:sensor_definitions prefix="${arm_prefix}" parent_link="world_frame"
-                x_val="-1.0414" y_val="0" z_val="1.18745" pitch="1.57" yaw="0" roll="0" />
-	<!-- end of sensor definitions -->
-	<joint name="world_to_stand" type="fixed">
-		<parent link="world_frame"/>
-		<child link="ur5_stand"/>
-		<origin xyz="-0.238 0 ${robot_stand_height * 0.5}"/>
-	</joint>
-	<joint name="world_to_base_padding" type="fixed">
-		<parent link="world_frame"/>
-		<child link="base_padding"/>
-		<origin xyz="-0.238 0 ${robot_stand_height}"/>
-	</joint>
-	<!-- end of arm-workcell link definitions -->
-	<!-- arm-workcell joint definitions -->
-	<joint name="stand_to_base" type="fixed">
-		<parent link="ur5_stand"/>
-		<child link="${arm_prefix}base_link"/>
-		<origin xyz="0 0 ${robot_stand_height * 0.5}" rpy="0 0 2.355"/>
-	</joint>
-	<!-- end of arm workcell joint definitions-->
-	<!-- arm-gripper coupling joint definitions -->
-	<joint name="${arm_prefix}to_gripper" type="fixed">
-		<parent link="${arm_prefix}ee_link"/>
-		<child link="${arm_prefix}gripper_frame"/>
-		<origin xyz="0 0 0" rpy="-1.57 0 -1.57"/> <!-- 0 1.57 0 -->
-	</joint>
-	<!-- end of arm-gripper coupling joint definitions -->
+    <xacro:include filename="$(find robot_config)/urdf/vacuum_gripper_macro.xacro"/>
+    <xacro:include filename="$(find robot_config)/urdf/ur5.urdf.xacro" />
+    <xacro:include filename="$(find robot_config)/urdf/workspace_components.xacro"/>
+    <xacro:include filename="$(find robot_config)/urdf/kinect_sensor_macro.xacro"/>
+    <!-- property list -->
+    <xacro:property name="workcell_height" value="1"/>
+    <xacro:property name="robot_stand_height" value="0.20"/>
+    <xacro:property name="vacuum_gripper_width" value="0.088"/>
+    <xacro:property name="attached_object_length" value="0.17"/>
+    <xacro:property name="attached_object_width" value="0.17"/>
+    <xacro:property name="attached_object_height" value="0.17"/>
+    <xacro:property name="arm_prefix" value=""/>
+    <!-- instantiating arm and gripper -->
+    <xacro:ur5_robot prefix="" joint_limited="true"/>
+    <xacro:vacuum_gripper_definition prefix="${arm_prefix}" gripper_adjustment="0.01"/>
+    <!-- instantiating workcell definitions -->
+    <xacro:workcell_zone2_components/>
+    <!-- end of workcell definitions -->
+    <!-- arm-workcell link definitions -->
+    <link name="ur5_stand">
+            <visual>
+                    <geometry>
+                            <cylinder radius="0.0735" length="${robot_stand_height}"/>
+                    </geometry>
+                    <material name="orange_transparent"/>
+            </visual>
+            <collision>
+                    <geometry>
+                            <cylinder radius="0.0735" length="${robot_stand_height}"/>
+                    </geometry>
+                    <material name="blue_transparent"/>
+            </collision>
+    </link>
+    <link name="base_padding">
+            <collision>
+                    <geometry>
+                            <cylinder radius="0.14" length="${robot_stand_height * 2}"/>
+                    </geometry>
+                    <material name="blue_transparent"/>
+            </collision>
+    </link>
+    <!-- instantiating sensor definitions -->
+    <xacro:sensor_definitions prefix="${arm_prefix}" parent_link="world_frame"
+            x_val="-1.0414" y_val="0" z_val="1.18745" pitch="1.57" yaw="0" roll="0" />
+    <!-- end of sensor definitions -->
+    <joint name="world_to_stand" type="fixed">
+            <parent link="world_frame"/>
+            <child link="ur5_stand"/>
+            <origin xyz="-0.238 0 ${robot_stand_height * 0.5}"/>
+    </joint>
+    <joint name="world_to_base_padding" type="fixed">
+            <parent link="world_frame"/>
+            <child link="base_padding"/>
+            <origin xyz="-0.238 0 ${robot_stand_height}"/>
+    </joint>
+    <!-- end of arm-workcell link definitions -->
+    <!-- arm-workcell joint definitions -->
+    <joint name="stand_to_base" type="fixed">
+            <parent link="ur5_stand"/>
+            <child link="${arm_prefix}base_link"/>
+            <origin xyz="0 0 ${robot_stand_height * 0.5}" rpy="0 0 2.355"/>
+    </joint>
+    <!-- end of arm workcell joint definitions-->
+    <!-- arm-gripper coupling joint definitions -->
+    <joint name="${arm_prefix}to_gripper" type="fixed">
+            <parent link="${arm_prefix}ee_link"/>
+            <child link="${arm_prefix}gripper_frame"/>
+            <origin xyz="0 0 0" rpy="-1.57 0 -1.57"/> <!-- 0 1.57 0 -->
+    </joint>
+    <!-- end of arm-gripper coupling joint definitions -->
 </robot>

Commit message: Bring training materials up-to-date
- latest auto-generated CMakeLists.txt/package.xml/MoveIt (Ex1-4 only)
- minor whitespace updates to match instruction code-fill
- tabs->spaces (in some files), for consistency
- sync solution_ws to template_ws

update deprecated calls
- MoveGroup -> MoveGroupInterface
- ExecuteKnownTrajectory service -> ExecuteTrajectory action
- some MoveIt params pushed to trajectory_execution namespace
- xacro.py -> xacro --inorder
- tf::Quaternion(r,p,y) -> tf::Quaternion(x,y,z,w)
- Eigen -> Eigen3
- add "xacro:" prefix where needed

- Ex3.4: add I-Beam.dae
- Ex4.1: match descartes path-size to match fake_ar_publisher marker size
- Ex4.1: change sign of corner coords to be more intuitive
- Ex4.1: re-instate "TODO" fill of AxialSymmetricPoint
- Ex4.2: add reference output files from each processing stage, move orig table.pcd file here
- demo1: remove .rosinstall (all in apt)
- demo1: fix print calls of pick/place pose to print positions (not function addr)
- demo1: fix load error in vaccuum_gripper...STL ("SOLID" keyword at file start)
- demo2: .rosinstall - remove universal_robot (use apt), update ur_modern_driver repo/branch
- demo2: fix hint-text for getNominalJointPose

Update exercise wiki pages
- convert leftover mediaWiki markup to GitHub markdown
- replace references to Eclipse/F3 with QTCreator/F2
- update links to current (kinetic), where available
- Ex3.3: add workaround to MoveIt Bug #955

Update Slides
- remove presentation date, chmod -x
- add/tweak content for clarity
- rework Slide 4 "Intro to Perception"
- remove "Introduction" slide (typically class-specific)

File: exercises/Perception-Driven_Manipulation/solution_ws/src/robot_config/urdf/ur5.urdf.xacro (robot description, xacro)
@@ -4,17 +4,17 @@
   <xacro:include filename="$(find ur_description)/urdf/ur.gazebo.xacro" />
   <!-- Inertia parameters -->
-  <property name="base_mass" value="4.0" />  <!-- This mass might be incorrect -->
-  <property name="shoulder_mass" value="3.7000" />
-  <property name="upper_arm_mass" value="8.3930" />
-  <property name="forearm_mass" value="2.2750" />
-  <property name="wrist_1_mass" value="1.2190" />
-  <property name="wrist_2_mass" value="1.2190" />
-  <property name="wrist_3_mass" value="0.1879" />
-  <property name="shoulder_cog" value="0.0 0.00193 -0.02561" />
-  <property name="upper_arm_cog" value="0.0 -0.024201 0.2125" />
-  <property name="forearm_cog" value="0.0 0.0265 0.11993" />
-  <property name="wrist_1_cog" value="0.0 0.110949 0.01634" />
-  <property name="wrist_2_cog" value="0.0 0.0018 0.11099" />
-  <property name="wrist_3_cog" value="0.0 0.001159 0.0" />
+  <xacro:property name="base_mass" value="4.0" />  <!-- This mass might be incorrect -->
+  <xacro:property name="shoulder_mass" value="3.7000" />
+  <xacro:property name="upper_arm_mass" value="8.3930" />
+  <xacro:property name="forearm_mass" value="2.2750" />
+  <xacro:property name="wrist_1_mass" value="1.2190" />
+  <xacro:property name="wrist_2_mass" value="1.2190" />
+  <xacro:property name="wrist_3_mass" value="0.1879" />
+  <xacro:property name="shoulder_cog" value="0.0 0.00193 -0.02561" />
+  <xacro:property name="upper_arm_cog" value="0.0 -0.024201 0.2125" />
+  <xacro:property name="forearm_cog" value="0.0 0.0265 0.11993" />
+  <xacro:property name="wrist_1_cog" value="0.0 0.110949 0.01634" />
+  <xacro:property name="wrist_2_cog" value="0.0 0.0018 0.11099" />
+  <xacro:property name="wrist_3_cog" value="0.0 0.001159 0.0" />
   <!-- Kinematic model -->
   <!-- Properties from urcontrol.conf -->
@@ -29,20 +29,20 @@
     center_of_mass = [ [0, -0.02561, 0.00193], [0.2125, 0, 0.11336], [0.11993, 0.0, 0.0265], [0, -0.0018, 0.01634], [0, 0.0018,0.01634], [0, 0, -0.001159] ]
   -->
-  <property name="ur5_d1" value="0.089159" />
-  <property name="ur5_a2" value="-0.42500" />
-  <property name="ur5_a3" value="-0.39225" />
-  <property name="ur5_d4" value="0.10915" />
-  <property name="ur5_d5" value="0.09465" />
-  <property name="ur5_d6" value="0.0823" />
+  <xacro:property name="ur5_d1" value="0.089159" />
+  <xacro:property name="ur5_a2" value="-0.42500" />
+  <xacro:property name="ur5_a3" value="-0.39225" />
+  <xacro:property name="ur5_d4" value="0.10915" />
+  <xacro:property name="ur5_d5" value="0.09465" />
+  <xacro:property name="ur5_d6" value="0.0823" />
   <!-- Arbitrary offsets for shoulder/elbow joints -->
-  <property name="shoulder_offset" value="0.13585" />  <!-- measured from model -->
-  <property name="elbow_offset" value="-0.1197" /> <!-- measured from model -->
+  <xacro:property name="shoulder_offset" value="0.13585" />  <!-- measured from model -->
+  <xacro:property name="elbow_offset" value="-0.1197" /> <!-- measured from model -->
   <!-- link lengths used in model -->
-  <property name="shoulder_height" value="${ur5_d1}" />
-  <property name="upper_arm_length" value="${-ur5_a2}" />
-  <property name="forearm_length" value="${-ur5_a3}" />
-  <property name="wrist_1_length" value="${ur5_d4 - elbow_offset - shoulder_offset}" />
-  <property name="wrist_2_length" value="${ur5_d5}" />
-  <property name="wrist_3_length" value="${ur5_d6}" />
+  <xacro:property name="shoulder_height" value="${ur5_d1}" />
+  <xacro:property name="upper_arm_length" value="${-ur5_a2}" />
+  <xacro:property name="forearm_length" value="${-ur5_a3}" />
+  <xacro:property name="wrist_1_length" value="${ur5_d4 - elbow_offset - shoulder_offset}" />
+  <xacro:property name="wrist_2_length" value="${ur5_d5}" />
+  <xacro:property name="wrist_3_length" value="${ur5_d6}" />
   <!--property name="shoulder_height" value="0.089159" /-->
   <!--property name="shoulder_offset" value="0.13585" /-->  <!-- shoulder_offset - elbow_offset + wrist_1_length = 0.10915 -->
@@ -53,13 +53,13 @@
   <!--property name="wrist_2_length" value="0.09465" /-->   <!-- In CAD this distance is 0.930, but in the spec it is 0.09465 -->
   <!--property name="wrist_3_length" value="0.0823" /-->
-  <property name="shoulder_radius" value="0.060" />   <!-- manually measured -->
-  <property name="upper_arm_radius" value="0.054" />  <!-- manually measured -->
-  <property name="elbow_radius" value="0.060" />      <!-- manually measured -->
-  <property name="forearm_radius" value="0.040" />    <!-- manually measured -->
-  <property name="wrist_radius" value="0.045" />      <!-- manually measured -->
+  <xacro:property name="shoulder_radius" value="0.060" />   <!-- manually measured -->
+  <xacro:property name="upper_arm_radius" value="0.054" />  <!-- manually measured -->
+  <xacro:property name="elbow_radius" value="0.060" />      <!-- manually measured -->
+  <xacro:property name="forearm_radius" value="0.040" />    <!-- manually measured -->
+  <xacro:property name="wrist_radius" value="0.045" />      <!-- manually measured -->
   <xacro:macro name="cylinder_inertial" params="radius length mass *origin">
     <inertial>
       <mass value="${mass}" />
-      <insert_block name="origin" />
+      <xacro:insert_block name="origin" />
       <inertia ixx="${0.0833333 * mass * (3 * radius * radius + length * length)}" ixy="0.0" ixz="0.0"
         iyy="${0.0833333 * mass * (3 * radius * radius + length * length)}" iyz="0.0"

File: exercises/Perception-Driven_Manipulation/solution_ws/src/robot_config/urdf/ur5_collision_avoidance.xacro (robot description, xacro)
@@ -25,4 +25,5 @@
                             <cylinder radius="0.0735" length="${robot_stand_height}"/>
                     </geometry>
+                    <material name="orange_transparent"/>
             </visual>
             <collision>
@@ -32,18 +33,4 @@
                     <material name="blue_transparent"/>
             </collision>
-    </link>
-    <link name="${arm_prefix}tool_interface_plate">
-        <visual>
-                <geometry>
-                        <box size="0.09525 0.09525 0.0127"/>
-                </geometry>
-                <material name="orange_transparent"/>
-        </visual>
-        <collision>
-                <geometry>
-                        <box size="0.09525 0.09525 0.0127"/>
-                </geometry>
-                <material name="blue_transparent"/>
-        </collision>
     </link>
     <link name="base_padding">
@@ -57,5 +44,5 @@
     <!-- instantiating sensor definitions -->
     <xacro:sensor_definitions prefix="${arm_prefix}" parent_link="world_frame"
-            x_val="-0.9208" y_val="-0.011125" z_val="1.21" pitch="1.57" yaw="0" roll="0" />
+            x_val="-1.0414" y_val="0" z_val="1.18745" pitch="1.57" yaw="0" roll="0" />
     <!-- end of sensor definitions -->
     <joint name="world_to_stand" type="fixed">
@@ -78,14 +65,8 @@
     <!-- end of arm workcell joint definitions-->
     <!-- arm-gripper coupling joint definitions -->
-    <joint name="${arm_prefix}to_interface_plate" type="fixed">
-            <parent link="${arm_prefix}ee_link"/>
-            <child link="${arm_prefix}tool_interface_plate"/>
-            <origin xyz="0.00635 0 0" rpy="0 1.57  0"/> <!-- 0 1.57 0 -->
-    </joint>
-    <!-- arm-gripper coupling joint definitions -->
     <joint name="${arm_prefix}to_gripper" type="fixed">
             <parent link="${arm_prefix}ee_link"/>
             <child link="${arm_prefix}gripper_frame"/>
-            <origin xyz="0.02 0 0" rpy="-1.57 0 -1.57"/> <!-- 0 1.57 0 -->
+            <origin xyz="0 0 0" rpy="-1.57 0 -1.57"/> <!-- 0 1.57 0 -->
     </joint>
     <!-- end of arm-gripper coupling joint definitions -->
