Commit message: update all ancillary folders in template workspace.  update calibration of camera parameters.

File: exercises/Perception-Driven_Manipulation/solution_ws/src/robot_config/urdf/ur5_collision_avoidance.xacro (robot description, xacro)
@@ -44,5 +44,5 @@
     <!-- instantiating sensor definitions -->
     <xacro:sensor_definitions prefix="${arm_prefix}" parent_link="world_frame"
-            x_val="-1.0414" y_val="0" z_val="1.18745" pitch="1.57" yaw="0" roll="0" />
+            x_val="-1.0732" y_val="-0.0397" z_val="1.2174" pitch="1.57" yaw="0" roll="0" />
     <!-- end of sensor definitions -->
     <joint name="world_to_stand" type="fixed">

File: exercises/Perception-Driven_Manipulation/template_ws/src/robot_config/urdf/ur5.urdf.xacro (robot description, xacro)
@@ -1,7 +1,6 @@
 <?xml version="1.0"?>
-<robot xmlns:xacro="http://www.ros.org/wiki/xacro">
-  <xacro:include filename="$(find ur_description)/urdf/ur5.transmission.xacro" />
-  <xacro:include filename="$(find ur_description)/urdf/ur5.gazebo.xacro" />
-  <property name="pi" value="3.14159265" />
+<robot xmlns:xacro="http://ros.org/wiki/xacro">
+  <xacro:include filename="$(find ur_description)/urdf/ur.transmission.xacro" />
+  <xacro:include filename="$(find ur_description)/urdf/ur.gazebo.xacro" />
   <!-- Inertia parameters -->
   <property name="base_mass" value="4.0" />  <!-- This mass might be incorrect -->
@@ -72,5 +71,5 @@
       <visual>
         <geometry>
-          <mesh filename="package://ur_description/meshes/ur5/visual/Base.dae" />
+          <mesh filename="package://ur_description/meshes/ur5/visual/base.dae" />
         </geometry>
         <material name="LightGrey">
@@ -103,5 +102,5 @@
       <visual>
         <geometry>
-          <mesh filename="package://ur_description/meshes/ur5/visual/Shoulder.dae" />
+          <mesh filename="package://ur_description/meshes/ur5/visual/shoulder.dae" />
         </geometry>
         <material name="LightGrey">
@@ -134,13 +133,13 @@
       <visual>
         <geometry>
-          <mesh filename="package://ur_description/meshes/ur5/visual/UpperArm.dae" />
-        </geometry>
-        <material name="LightGrey">
-          <color rgba="0.7 0.7 0.7 1.0"/>
-        </material>
-      </visual>
-      <collision>
-        <geometry>
-          <mesh filename="package://ur_description/meshes/ur5/collision/upper_arm.stl" />
+          <mesh filename="package://ur_description/meshes/ur5/visual/upperarm.dae" />
+        </geometry>
+        <material name="LightGrey">
+          <color rgba="0.7 0.7 0.7 1.0"/>
+        </material>
+      </visual>
+      <collision>
+        <geometry>
+          <mesh filename="package://ur_description/meshes/ur5/collision/upperarm.stl" />
         </geometry>
       </collision>
@@ -165,5 +164,5 @@
       <visual>
         <geometry>
-          <mesh filename="package://ur_description/meshes/ur5/visual/Forearm.dae" />
+          <mesh filename="package://ur_description/meshes/ur5/visual/forearm.dae" />
         </geometry>
         <material name="LightGrey">
@@ -196,13 +195,13 @@
       <visual>
         <geometry>
-          <mesh filename="package://ur_description/meshes/ur5/visual/Wrist1.dae" />
-        </geometry>
-        <material name="LightGrey">
-          <color rgba="0.7 0.7 0.7 1.0"/>
-        </material>
-      </visual>
-      <collision>
-        <geometry>
-          <mesh filename="package://ur_description/meshes/ur5/collision/wrist_1.stl" />
+          <mesh filename="package://ur_description/meshes/ur5/visual/wrist1.dae" />
+        </geometry>
+        <material name="LightGrey">
+          <color rgba="0.7 0.7 0.7 1.0"/>
+        </material>
+      </visual>
+      <collision>
+        <geometry>
+          <mesh filename="package://ur_description/meshes/ur5/collision/wrist1.stl" />
         </geometry>
       </collision>
@@ -227,13 +226,13 @@
       <visual>
         <geometry>
-          <mesh filename="package://ur_description/meshes/ur5/visual/Wrist2.dae" />
-        </geometry>
-        <material name="LightGrey">
-          <color rgba="0.7 0.7 0.7 1.0"/>
-        </material>
-      </visual>
-      <collision>
-        <geometry>
-          <mesh filename="package://ur_description/meshes/ur5/collision/wrist_2.stl" />
+          <mesh filename="package://ur_description/meshes/ur5/visual/wrist2.dae" />
+        </geometry>
+        <material name="LightGrey">
+          <color rgba="0.7 0.7 0.7 1.0"/>
+        </material>
+      </visual>
+      <collision>
+        <geometry>
+          <mesh filename="package://ur_description/meshes/ur5/collision/wrist2.stl" />
         </geometry>
       </collision>
@@ -258,13 +257,13 @@
       <visual>
         <geometry>
-          <mesh filename="package://ur_description/meshes/ur5/visual/Wrist3.dae" />
-        </geometry>
-        <material name="LightGrey">
-          <color rgba="0.7 0.7 0.7 1.0"/>
-        </material>
-      </visual>
-      <collision>
-        <geometry>
-          <mesh filename="package://ur_description/meshes/ur5/collision/wrist_3.stl" />
+          <mesh filename="package://ur_description/meshes/ur5/visual/wrist3.dae" />
+        </geometry>
+        <material name="LightGrey">
+          <color rgba="0.7 0.7 0.7 1.0"/>
+        </material>
+      </visual>
+      <collision>
+        <geometry>
+          <mesh filename="package://ur_description/meshes/ur5/collision/wrist3.stl" />
         </geometry>
       </collision>
@@ -286,6 +285,6 @@
       </collision>
     </link>
-    <xacro:ur5_arm_transmission prefix="${prefix}" />
-    <xacro:ur5_arm_gazebo prefix="${prefix}" />
+    <xacro:ur_arm_transmission prefix="${prefix}" />
+    <xacro:ur_arm_gazebo prefix="${prefix}" />
   </xacro:macro>
 </robot>

File: exercises/Perception-Driven_Manipulation/template_ws/src/robot_config/urdf/ur5_collision_avoidance.xacro (robot description, xacro)
@@ -1,73 +1,73 @@
 <?xml version="1.0" ?>
 <robot name="ur5_collision_avoidance" xmlns:xacro="http://ros.org/wiki/xacro">
-	<xacro:include filename="$(find robot_config)/urdf/vacuum_gripper_macro.xacro"/>
-  <xacro:include filename="$(find robot_config)/urdf/ur5.urdf.xacro" />
-	<xacro:include filename="$(find robot_config)/urdf/workspace_components.xacro"/>
-	<xacro:include filename="$(find robot_config)/urdf/kinect_sensor_macro.xacro"/>
-	<!-- property list -->
-	<xacro:property name="workcell_height" value="1"/>
-	<xacro:property name="robot_stand_height" value="0.20"/>
-	<xacro:property name="vacuum_gripper_width" value="0.088"/>
-        <xacro:property name="attached_object_length" value="0.17"/>
-	<xacro:property name="attached_object_width" value="0.17"/>
-	<xacro:property name="attached_object_height" value="0.17"/>
-	<xacro:property name="arm_prefix" value=""/>
-	<!-- instantiating arm and gripper -->
-  <xacro:ur5_robot prefix="" joint_limited="true"/>
-	<xacro:vacuum_gripper_definition prefix="${arm_prefix}" gripper_adjustment="0.01"/>
-	<!-- instantiating workcell definitions -->
-	<xacro:workcell_zone2_components/>
-	<!-- end of workcell definitions -->
-	<!-- arm-workcell link definitions -->
-	<link name="ur5_stand">
-		<visual>
-			<geometry>
-				<cylinder radius="0.0735" length="${robot_stand_height}"/>
-			</geometry>
-			<material name="orange_transparent"/>
-		</visual>
-		<collision>
-			<geometry>
-				<cylinder radius="0.0735" length="${robot_stand_height}"/>
-			</geometry>
-			<material name="blue_transparent"/>
-		</collision>
-	</link>
-	<link name="base_padding">
-		<collision>
-			<geometry>
-				<cylinder radius="0.14" length="${robot_stand_height * 2}"/>
-			</geometry>
-			<material name="blue_transparent"/>
-		</collision>
-	</link>
-	<!-- instantiating sensor definitions -->
-	<xacro:sensor_definitions prefix="${arm_prefix}" parent_link="ur5_stand"
-		x_val="-0.981" y_val="0.190" z_val="1.015" pitch="1.145" yaw="0.035" roll="0.019" />
-	<!-- end of sensor definitions -->
-	<joint name="world_to_stand" type="fixed">
-		<parent link="world_frame"/>
-		<child link="ur5_stand"/>
-		<origin xyz="-0.238 0 ${robot_stand_height * 0.5}"/>
-	</joint>
-	<joint name="world_to_base_padding" type="fixed">
-		<parent link="world_frame"/>
-		<child link="base_padding"/>
-		<origin xyz="-0.238 0 ${robot_stand_height}"/>
-	</joint>
-	<!-- end of arm-workcell link definitions -->
-	<!-- arm-workcell joint definitions -->
-	<joint name="stand_to_base" type="fixed">
-		<parent link="ur5_stand"/>
-		<child link="${arm_prefix}base_link"/>
-		<origin xyz="0 0 ${robot_stand_height * 0.5}" rpy="0 0 2.355"/>
-	</joint>
-	<!-- end of arm workcell joint definitions-->
-	<!-- arm-gripper coupling joint definitions -->
-	<joint name="${arm_prefix}to_gripper" type="fixed">
-		<parent link="${arm_prefix}ee_link"/>
-		<child link="${arm_prefix}gripper_frame"/>
-		<origin xyz="0 0 0" rpy="-1.57 0 -1.57"/> <!-- 0 1.57 0 -->
-	</joint>
-	<!-- end of arm-gripper coupling joint definitions -->
+    <xacro:include filename="$(find robot_config)/urdf/vacuum_gripper_macro.xacro"/>
+    <xacro:include filename="$(find robot_config)/urdf/ur5.urdf.xacro" />
+    <xacro:include filename="$(find robot_config)/urdf/workspace_components.xacro"/>
+    <xacro:include filename="$(find robot_config)/urdf/kinect_sensor_macro.xacro"/>
+    <!-- property list -->
+    <xacro:property name="workcell_height" value="1"/>
+    <xacro:property name="robot_stand_height" value="0.20"/>
+    <xacro:property name="vacuum_gripper_width" value="0.088"/>
+    <xacro:property name="attached_object_length" value="0.17"/>
+    <xacro:property name="attached_object_width" value="0.17"/>
+    <xacro:property name="attached_object_height" value="0.17"/>
+    <xacro:property name="arm_prefix" value=""/>
+    <!-- instantiating arm and gripper -->
+    <xacro:ur5_robot prefix="" joint_limited="true"/>
+    <xacro:vacuum_gripper_definition prefix="${arm_prefix}" gripper_adjustment="0.01"/>
+    <!-- instantiating workcell definitions -->
+    <xacro:workcell_zone2_components/>
+    <!-- end of workcell definitions -->
+    <!-- arm-workcell link definitions -->
+    <link name="ur5_stand">
+            <visual>
+                    <geometry>
+                            <cylinder radius="0.0735" length="${robot_stand_height}"/>
+                    </geometry>
+                    <material name="orange_transparent"/>
+            </visual>
+            <collision>
+                    <geometry>
+                            <cylinder radius="0.0735" length="${robot_stand_height}"/>
+                    </geometry>
+                    <material name="blue_transparent"/>
+            </collision>
+    </link>
+    <link name="base_padding">
+            <collision>
+                    <geometry>
+                            <cylinder radius="0.14" length="${robot_stand_height * 2}"/>
+                    </geometry>
+                    <material name="blue_transparent"/>
+            </collision>
+    </link>
+    <!-- instantiating sensor definitions -->
+    <xacro:sensor_definitions prefix="${arm_prefix}" parent_link="world_frame"
+            x_val="-1.0414" y_val="0" z_val="1.18745" pitch="1.57" yaw="0" roll="0" />
+    <!-- end of sensor definitions -->
+    <joint name="world_to_stand" type="fixed">
+            <parent link="world_frame"/>
+            <child link="ur5_stand"/>
+            <origin xyz="-0.238 0 ${robot_stand_height * 0.5}"/>
+    </joint>
+    <joint name="world_to_base_padding" type="fixed">
+            <parent link="world_frame"/>
+            <child link="base_padding"/>
+            <origin xyz="-0.238 0 ${robot_stand_height}"/>
+    </joint>
+    <!-- end of arm-workcell link definitions -->
+    <!-- arm-workcell joint definitions -->
+    <joint name="stand_to_base" type="fixed">
+            <parent link="ur5_stand"/>
+            <child link="${arm_prefix}base_link"/>
+            <origin xyz="0 0 ${robot_stand_height * 0.5}" rpy="0 0 2.355"/>
+    </joint>
+    <!-- end of arm workcell joint definitions-->
+    <!-- arm-gripper coupling joint definitions -->
+    <joint name="${arm_prefix}to_gripper" type="fixed">
+            <parent link="${arm_prefix}ee_link"/>
+            <child link="${arm_prefix}gripper_frame"/>
+            <origin xyz="0 0 0" rpy="-1.57 0 -1.57"/> <!-- 0 1.57 0 -->
+    </joint>
+    <!-- end of arm-gripper coupling joint definitions -->
 </robot>

Commit message: tested and working, picking up boxes.

File: exercises/Perception-Driven_Manipulation/solution_ws/src/robot_config/urdf/ur5_collision_avoidance.xacro (robot description, xacro)
@@ -25,5 +25,4 @@
                             <cylinder radius="0.0735" length="${robot_stand_height}"/>
                     </geometry>
-                    <material name="orange_transparent"/>
             </visual>
             <collision>
@@ -33,4 +32,18 @@
                     <material name="blue_transparent"/>
             </collision>
+    </link>
+    <link name="${arm_prefix}tool_interface_plate">
+        <visual>
+                <geometry>
+                        <box size="0.09525 0.09525 0.0127"/>
+                </geometry>
+                <material name="orange_transparent"/>
+        </visual>
+        <collision>
+                <geometry>
+                        <box size="0.09525 0.09525 0.0127"/>
+                </geometry>
+                <material name="blue_transparent"/>
+        </collision>
     </link>
     <link name="base_padding">
@@ -44,5 +57,5 @@
     <!-- instantiating sensor definitions -->
     <xacro:sensor_definitions prefix="${arm_prefix}" parent_link="world_frame"
-            x_val="-1.0732" y_val="-0.0397" z_val="1.2174" pitch="1.57" yaw="0" roll="0" />
+            x_val="-0.9208" y_val="-0.011125" z_val="1.21" pitch="1.57" yaw="0" roll="0" />
     <!-- end of sensor definitions -->
     <joint name="world_to_stand" type="fixed">
@@ -65,8 +78,14 @@
     <!-- end of arm workcell joint definitions-->
     <!-- arm-gripper coupling joint definitions -->
+    <joint name="${arm_prefix}to_interface_plate" type="fixed">
+            <parent link="${arm_prefix}ee_link"/>
+            <child link="${arm_prefix}tool_interface_plate"/>
+            <origin xyz="0.00635 0 0" rpy="0 1.57  0"/> <!-- 0 1.57 0 -->
+    </joint>
+    <!-- arm-gripper coupling joint definitions -->
     <joint name="${arm_prefix}to_gripper" type="fixed">
             <parent link="${arm_prefix}ee_link"/>
             <child link="${arm_prefix}gripper_frame"/>
-            <origin xyz="0 0 0" rpy="-1.57 0 -1.57"/> <!-- 0 1.57 0 -->
+            <origin xyz="0.02 0 0" rpy="-1.57 0 -1.57"/> <!-- 0 1.57 0 -->
     </joint>
     <!-- end of arm-gripper coupling joint definitions -->

Commit message: updated xacro to comply with current universal robot macro xacro

File: exercises/Perception-Driven_Manipulation/solution_ws/src/robot_config/urdf/ur5_collision_avoidance.xacro (robot description, xacro)
@@ -2,5 +2,5 @@
 <robot name="ur5_collision_avoidance" xmlns:xacro="http://ros.org/wiki/xacro">
     <xacro:include filename="$(find robot_config)/urdf/vacuum_gripper_macro.xacro"/>
-    <xacro:include filename="$(find ur_description)/urdf/ur5.urdf.xacro" />
+    <xacro:include filename="$(find ur_description)/urdf/ur_macro.xacro" />
     <xacro:include filename="$(find robot_config)/urdf/workspace_components.xacro"/>
     <xacro:include filename="$(find robot_config)/urdf/kinect_sensor_macro.xacro"/>
@@ -14,5 +14,25 @@
     <xacro:property name="arm_prefix" value=""/>
     <!-- instantiating arm and gripper -->
-    <xacro:ur5_robot prefix="" joint_limited="true"/>
+       <!-- parameters -->
+    <xacro:arg name="ur_type" default="ur5"/>
+    <xacro:arg name="joint_limit_params" default="$(find ur_description)/config/$(arg ur_type)/joint_limits.yaml"/>
+    <xacro:arg name="kinematics_params" default="$(find ur_description)/config/$(arg ur_type)/default_kinematics.yaml"/>
+    <xacro:arg name="physical_params" default="$(find ur_description)/config/$(arg ur_type)/physical_parameters.yaml"/>
+    <xacro:arg name="visual_params" default="$(find ur_description)/config/$(arg ur_type)/visual_parameters.yaml"/>
+    <xacro:arg name="transmission_hw_interface" default="hardware_interface/PositionJointInterface"/>
+    <xacro:arg name="safety_limits" default="false"/>
+    <xacro:arg name="safety_pos_margin" default="0.15"/>
+    <xacro:arg name="safety_k_position" default="20"/>
+    <xacro:ur_robot
+     prefix=""
+     joint_limits_parameters_file="$(arg joint_limit_params)"
+     kinematics_parameters_file="$(arg kinematics_params)"
+     physical_parameters_file="$(arg physical_params)"
+     visual_parameters_file="$(arg visual_params)"
+     transmission_hw_interface="$(arg transmission_hw_interface)"
+     safety_limits="$(arg safety_limits)"
+     safety_pos_margin="$(arg safety_pos_margin)"
+     safety_k_position="$(arg safety_k_position)"/>
+    <!-- instantiating arm and gripper -->
     <xacro:vacuum_gripper_definition prefix="${arm_prefix}" gripper_adjustment="0.01"/>
     <!-- instantiating workcell definitions -->
@@ -65,8 +85,8 @@
     <!-- end of arm workcell joint definitions-->
     <!-- arm-gripper coupling joint definitions -->
-    <joint name="${arm_prefix}to_gripper" type="fixed">
-            <parent link="${arm_prefix}ee_link"/>
+    <joint name="${arm_prefix}wrist_to_gripper" type="fixed">
+            <parent link="${arm_prefix}tool0"/>
             <child link="${arm_prefix}gripper_frame"/>
-            <origin xyz="0 0 0" rpy="-1.57 0 -1.57"/> <!-- 0 1.57 0 -->
+            <origin xyz="0 0 0" rpy="0 0 0"/> <!-- 0 1.57 0 -->
     </joint>
     <!-- end of arm-gripper coupling joint definitions -->
