Commit message: Add advanced descartes puzzle exercise

File: exercises/5.0/src/myworkcell_support/urdf/workcell.xacro (robot description, xacro)
@@ -2,4 +2,7 @@
 <robot name="myworkcell" xmlns:xacro="http://ros.org/wiki/xacro">
   <xacro:include filename="$(find ur_description)/urdf/ur5.urdf.xacro" />
+  <!-- This contains the macro "ses_part_macro" that places the clip wrt the tool tip -->
+  <include filename="$(find myworkcell_support)/urdf/puzzle_mount.xacro" />
+  <include filename="$(find myworkcell_support)/urdf/grinder.xacro" />
   <link name="world"/>
   <link name="table">
@@ -22,4 +25,9 @@
     <origin xyz="0 0 0.5" rpy="0 0 0"/>
   </joint>
+  <joint name="world_to_grinder" type="fixed">
+    <parent link="world"/>
+    <child link="grinder_frame"/>
+    <origin xyz="0.0 -0.4 0.6" rpy="0 3.14159 0"/>
+  </joint>
   <joint name="world_to_camera" type="fixed">
     <parent link="world"/>
@@ -32,3 +40,8 @@
     <origin xyz="0 0 0" rpy="0 0 0"/>
   </joint>
+  <joint name="robot_tool" type="fixed">
+    <parent link="tool0"/>
+    <child link="ee_mount"/>
+    <origin xyz="0 0 0" rpy="1.5708 0 0"/>
+  </joint>
 </robot>

Commit message: Update advanced exercises
- update CMakeLists/package.xml to latest templates
- clean up minor whitespace inconsistencies
- fix misc warnings (e.g. Eigen3, missing xacro: prefix)
- move Perception to Exercise 5.1, to match wiki
- Move STOMP to Exercise 5.2, to match wiki
- add new Exercise 5.4: python/OpenCV
- update instructions for Ex 5.0, 5.1, 5.4, 6.1

File: exercises/5.0/src/myworkcell_support/urdf/workcell.xacro (robot description, xacro)
@@ -2,7 +2,6 @@
 <robot name="myworkcell" xmlns:xacro="http://ros.org/wiki/xacro">
   <xacro:include filename="$(find ur_description)/urdf/ur5.urdf.xacro" />
-  <!-- This contains the macro "ses_part_macro" that places the clip wrt the tool tip -->
-  <include filename="$(find myworkcell_support)/urdf/puzzle_mount.xacro" />
-  <include filename="$(find myworkcell_support)/urdf/grinder.xacro" />
+  <xacro:include filename="$(find myworkcell_support)/urdf/grinder.xacro" />
+  <xacro:include filename="$(find myworkcell_support)/urdf/puzzle_mount.xacro" />
   <link name="world"/>
   <link name="table">
@@ -25,9 +24,4 @@
     <origin xyz="0 0 0.5" rpy="0 0 0"/>
   </joint>
-  <joint name="world_to_grinder" type="fixed">
-    <parent link="world"/>
-    <child link="grinder_frame"/>
-    <origin xyz="0.0 -0.4 0.6" rpy="0 3.14159 0"/>
-  </joint>
   <joint name="world_to_camera" type="fixed">
     <parent link="world"/>
@@ -40,5 +34,10 @@
     <origin xyz="0 0 0" rpy="0 0 0"/>
   </joint>
-  <joint name="robot_tool" type="fixed">
+  <joint name="world_to_grinder" type="fixed">
+    <parent link="world"/>
+    <child link="grinder_frame"/>
+    <origin xyz="0 -0.4 0.6" rpy="0 3.14159 0"/>
+  </joint>
+  <joint name="tool_to_puzzle" type="fixed">
     <parent link="tool0"/>
     <child link="ee_mount"/>
