Commit message: fixup

File: exercises/Perception-Driven_Manipulation/solution_ws/src/robot_workcell_support/urdf/ur5_collision_avoidance.xacro (robot description, xacro)
@@ -1,8 +1,8 @@
 <?xml version="1.0" ?>
 <robot name="ur5_collision_avoidance" xmlns:xacro="http://ros.org/wiki/xacro">
-    <xacro:include filename="$(find robot_config)/urdf/vacuum_gripper_macro.xacro"/>
+    <xacro:include filename="$(find robot_workcell_support)/urdf/vacuum_gripper_macro.xacro"/>
     <xacro:include filename="$(find ur_description)/urdf/ur5.urdf.xacro" />
-    <xacro:include filename="$(find robot_config)/urdf/workspace_components.xacro"/>
-    <xacro:include filename="$(find robot_config)/urdf/kinect_sensor_macro.xacro"/>
+    <xacro:include filename="$(find robot_workcell_support)/urdf/workspace_components.xacro"/>
+    <xacro:include filename="$(find robot_workcell_support)/urdf/kinect_sensor_macro.xacro"/>
     <!-- property list -->
     <xacro:property name="workcell_height" value="1"/>

File: exercises/Perception-Driven_Manipulation/solution_ws/src/robot_workcell_support/urdf/vacuum_gripper_macro.xacro (robot description, xacro)
@@ -16,5 +16,5 @@
 				<origin xyz="0 0 -0.048" rpy="0 0 0"/>
 				<geometry>
-					<mesh filename="package://robot_config/meshes/vacuum_gripper_single_suction_cup.STL" />
+					<mesh filename="package://robot_workcell_support/meshes/vacuum_gripper_single_suction_cup.STL" />
 				</geometry>
 				<material name="silver">
