Commit message: minor tweaks to the urdf to be in compliance with the UR xacro

File: exercises/Perception-Driven_Manipulation/solution_ws/src/robot_workcell_support/urdf/ur5_workcell.xacro (robot description, xacro)
@@ -2,5 +2,4 @@
 <robot name="ur5_workcell" xmlns:xacro="http://ros.org/wiki/xacro">
     <xacro:include filename="$(find robot_workcell_support)/urdf/vacuum_gripper_macro.xacro"/>
-    <!-- xacro:include filename="$(find ur_description)/urdf/ur.urdf.xacro" /> -->
     <xacro:include filename="$(find ur_description)/urdf/ur_macro.xacro"/>
     <xacro:include filename="$(find robot_workcell_support)/urdf/workspace_components.xacro"/>
@@ -15,9 +14,7 @@
     <xacro:property name="arm_prefix" value=""/>
     <!-- instantiating robot arm and gripper -->
-    <!-- <xacro:ur5_robot prefix="" joint_limited="true"/> -->
-    <!-- parameters -->
+    <!-- ur parameters -->
+    <xacro:arg name="prefix" default="${arm_prefix}"/><!-- Remove once PR https://github.com/UniversalRobots/Universal_Robots_ROS2_Driver/pull/149 is merged-->
     <xacro:arg name="ur_type" default="ur5"/>
-    <xacro:arg name="prefix" default=""/>
-    <xacro:arg name="joint_limit_params" default="$(find ur_description)/config/$(arg ur_type)/joint_limits.yaml"/>
     <xacro:arg name="joint_limit_params" default="$(find ur_description)/config/$(arg ur_type)/joint_limits.yaml"/>
     <xacro:arg name="kinematics_params" default="$(find ur_description)/config/$(arg ur_type)/default_kinematics.yaml"/>
@@ -29,9 +26,9 @@
 		<xacro:arg name="safety_k_position" default="20"/>
 		<!-- ros2_control related parameters -->
-		<xacro:arg name="use_fake_hardware" default="false" />
+		<xacro:arg name="use_fake_hardware" default="true" />
 		<xacro:arg name="fake_sensor_commands" default="false" />
-   <!-- arm -->
+   <!-- ur arm instantiation -->
    <xacro:ur_robot
-     prefix=""
+     prefix="${arm_prefix}"
      joint_limits_parameters_file="$(arg joint_limit_params)"
      kinematics_parameters_file="$(arg kinematics_params)"
@@ -95,6 +92,6 @@
     <!-- end of arm workcell joint definitions-->
     <!-- arm-gripper coupling joint definitions -->
-    <joint name="${arm_prefix}to_gripper" type="fixed">
-            <parent link="${arm_prefix}ee_link"/>
+    <joint name="${arm_prefix}wrist_to_gripper" type="fixed">
+            <parent link="${arm_prefix}tool0"/>
             <child link="${arm_prefix}gripper_frame"/>
             <origin xyz="0 0 0" rpy="-1.57 0 -1.57"/> <!-- 0 1.57 0 -->

Commit message: added argument for taking init positions joint files

File: exercises/Perception-Driven_Manipulation/solution_ws/src/robot_workcell_support/urdf/ur5_workcell.xacro (robot description, xacro)
@@ -21,5 +21,5 @@
     <xacro:arg name="physical_params" default="$(find ur_description)/config/$(arg ur_type)/physical_parameters.yaml"/>
     <xacro:arg name="visual_params" default="$(find ur_description)/config/$(arg ur_type)/visual_parameters.yaml"/>
-		<xacro:arg name="transmission_hw_interface" default="blah"/>
+		<xacro:arg name="transmission_hw_interface" default=""/>
 		<xacro:arg name="safety_limits" default="false"/>
 		<xacro:arg name="safety_pos_margin" default="0.15"/>
@@ -28,4 +28,13 @@
 		<xacro:arg name="use_fake_hardware" default="true" />
 		<xacro:arg name="fake_sensor_commands" default="false" />
+		<!-- ros2 fake_components/generic_system  initial joints -->
+		<xacro:arg name="initial_positions_file" default=""/>
+		<xacro:property name="initial_positions_file_" value="$(arg initial_positions_file)"/>
+		<xacro:if value="${initial_positions_file_ == ''}">
+		  <xacro:property name="initial_positions" value="${dict(shoulder_pan_joint=0,shoulder_lift_joint=-1.57,elbow_joint=0,wrist_1_joint=-1.57,wrist_2_joint=0.0,wrist_3_joint=0.0)}" />
+		</xacro:if>
+		<xacro:if value="${initial_positions_file_ != ''}">
+		  <xacro:property name="initial_positions" value="${load_yaml(initial_positions_file_)}"/>
+		</xacro:if>
    <!-- ur arm instantiation -->
    <xacro:ur_robot
@@ -40,5 +49,6 @@
      safety_k_position="$(arg safety_k_position)"
      use_fake_hardware="$(arg use_fake_hardware)"
-     fake_sensor_commands="$(arg fake_sensor_commands)" />
+     fake_sensor_commands="$(arg fake_sensor_commands)"
+     initial_positions="${initial_positions}" />
     <!-- instantiating robot arm and gripper -->
     <xacro:vacuum_gripper_definition prefix="${arm_prefix}" gripper_adjustment="0.01"/>

Commit message: capturing working state of pick and place application, needs cleanup and updates to instructional comments

File: exercises/Perception-Driven_Manipulation/solution_ws/src/robot_workcell_support/urdf/ur5_workcell.xacro (robot description, xacro)
@@ -105,5 +105,5 @@
             <parent link="${arm_prefix}tool0"/>
             <child link="${arm_prefix}gripper_frame"/>
-            <origin xyz="0 0 0" rpy="-1.57 0 -1.57"/> <!-- 0 1.57 0 -->
+            <origin xyz="0 0 0" rpy="0 0 0"/> <!-- 0 1.57 0 -->
     </joint>
     <!-- end of arm-gripper coupling joint definitions -->

Commit message: minor changes to limit joint ranges and improve motion planning

File: exercises/Perception-Driven_Manipulation/solution_ws/src/robot_workcell_support/urdf/ur5_workcell.xacro (robot description, xacro)
@@ -21,20 +21,21 @@
     <xacro:arg name="physical_params" default="$(find ur_description)/config/$(arg ur_type)/physical_parameters.yaml"/>
     <xacro:arg name="visual_params" default="$(find ur_description)/config/$(arg ur_type)/visual_parameters.yaml"/>
-		<xacro:arg name="transmission_hw_interface" default=""/>
-		<xacro:arg name="safety_limits" default="false"/>
-		<xacro:arg name="safety_pos_margin" default="0.15"/>
-		<xacro:arg name="safety_k_position" default="20"/>
-		<!-- ros2_control related parameters -->
-		<xacro:arg name="use_fake_hardware" default="true" />
-		<xacro:arg name="fake_sensor_commands" default="false" />
-		<!-- ros2 fake_components/generic_system  initial joints -->
-		<xacro:arg name="initial_positions_file" default=""/>
-		<xacro:property name="initial_positions_file_" value="$(arg initial_positions_file)"/>
-		<xacro:if value="${initial_positions_file_ == ''}">
-		  <xacro:property name="initial_positions" value="${dict(shoulder_pan_joint=0,shoulder_lift_joint=-1.57,elbow_joint=0,wrist_1_joint=-1.57,wrist_2_joint=0.0,wrist_3_joint=0.0)}" />
-		</xacro:if>
-		<xacro:if value="${initial_positions_file_ != ''}">
-		  <xacro:property name="initial_positions" value="${load_yaml(initial_positions_file_)}"/>
-		</xacro:if>
+	<xacro:arg name="transmission_hw_interface" default=""/>
+	<xacro:arg name="safety_limits" default="false"/>
+	<xacro:arg name="safety_pos_margin" default="0.15"/>
+	<xacro:arg name="safety_k_position" default="20"/>
+	<!-- ros2_control related parameters -->
+	<xacro:arg name="use_fake_hardware" default="true" />
+	<xacro:arg name="fake_sensor_commands" default="false" />
+	<xacro:arg name="robot_ip" default="10.0.1.186"/>
+	<!-- ros2 fake_components/generic_system  initial joints -->
+	<xacro:arg name="initial_positions_file" default=""/>
+	<xacro:property name="initial_positions_file_" value="$(arg initial_positions_file)"/>
+	<xacro:if value="${initial_positions_file_ == ''}">
+	  <xacro:property name="initial_positions" value="${dict(shoulder_pan_joint=0,shoulder_lift_joint=-1.57,elbow_joint=0,wrist_1_joint=-1.57,wrist_2_joint=0.0,wrist_3_joint=0.0)}" />
+	</xacro:if>
+	<xacro:if value="${initial_positions_file_ != ''}">
+	  <xacro:property name="initial_positions" value="${load_yaml(initial_positions_file_)}"/>
+	</xacro:if>
    <!-- ur arm instantiation -->
    <xacro:ur_robot

File: exercises/Perception-Driven_Manipulation/solution_ws/src/robot_workcell_support/urdf/vacuum_gripper_macro.xacro (robot description, xacro)
@@ -41,9 +41,4 @@
 				</material>
 			</visual>
-			<collision>
-				<geometry>
-					<sphere radius="0.005"/>
-				</geometry>
-			</collision>
 		</link>
 		<joint name="${prefix}gripper_to_palm" type="fixed">
