Commit message: 3.0 no changes. 3.1 to humble

File: exercises/3.1/ros2/src/myworkcell_support/urdf/workcell.urdf.xacro (robot description, xacro)
@@ -7,5 +7,7 @@
   <xacro:arg name="fake_sensor_commands" default="true"/>
   <xacro:ur_robot
+      name="my_ur5"
       prefix=""
+      parent="table"
       joint_limits_parameters_file="$(find ur_description)/config/$(arg ur_type)/joint_limits.yaml"
       kinematics_parameters_file="$(find ur_description)/config/$(arg ur_type)/default_kinematics.yaml"
@@ -13,5 +15,7 @@
       visual_parameters_file="$(find ur_description)/config/$(arg ur_type)/visual_parameters.yaml"
       use_fake_hardware="$(arg use_fake_hardware)"
-      fake_sensor_commands="$(arg fake_sensor_commands)"/>
+      fake_sensor_commands="$(arg fake_sensor_commands)">
+    <origin xyz="0 0 0" rpy="0 0 0"/>
+  </xacro:ur_robot>
   <link name="world"/>
   <link name="table">
@@ -33,9 +37,4 @@
     <origin xyz="0 0 0.5" rpy="0 0 0"/>
   </joint>
-  <joint name="table_to_robot" type="fixed">
-    <parent link="table"/>
-    <child link="base_link"/>
-    <origin xyz="0 0 0" rpy="0 0 0"/>
-  </joint>
   <joint name="world_to_camera" type="fixed">
     <parent link="world"/>
