Commit message: Calibration instruction fixes

File: exercises/9.0/template/cal_demo_support/urdf/workcell.urdf.xacro (robot description, xacro)
@@ -15,12 +15,10 @@
   <parent link="tool0"/>
   <child link="target"/>
-  <origin xyz="0.055784058339184643 0.11487059843451272 0.20165459507523578"
-    rpy="-0.17356982424404177 1.5097766327158793 2.1768171924570656"/>
+  <origin xyz="0 0 0" rpy="0 0 0"/>
 </joint>
 <joint name="base_to_camera" type="fixed">
   <parent link="base_link"/>
   <child link="camera"/>
-  <origin xyz="-0.020595376784745552 1.2683438657723451 0.28518860273351132"
-    rpy="-1.1843479510784112 0.10553100089290253 3.1306767554292696"/>
+  <origin xyz="0 0 0" rpy="0 0 0"/>
 </joint>
 </robot>
