Commit message: fixed joint_state_broadcaster for the Perception template demo, added no collision between shoulder_link and base_link_interia

File: exercises/Perception-Driven_Manipulation/ros2/template_ws/src/robot_workcell_support/urdf/ur5_workcell.xacro (robot description, xacro)
@@ -106,4 +106,9 @@
             <origin xyz="0 0 0" rpy="0 0 0"/> <!-- 0 1.57 0 -->
     </joint>
+    <joint name="world_frame_to_world" type="fixed">
+            <parent link="world_frame"/>
+            <child link="world"/>
+            <origin xyz="0 0 0" rpy="0 0 0"/>
+    </joint>
     <!-- end of arm-gripper coupling joint definitions -->
 </robot>
