Commit message: Attempt to fix Perception lab

File: exercises/Perception-Driven_Manipulation/ros2/solution_ws/src/robot_workcell_support/urdf/ur5_workcell.xacro (robot description, xacro)
@@ -40,5 +40,7 @@
    <!-- ur arm instantiation -->
    <xacro:ur_robot
-     prefix="${arm_prefix}"
+     name="ur5"
+     tf_prefix="${arm_prefix}"
+     parent="ur5_stand"
      joint_limits_parameters_file="$(arg joint_limit_params)"
      kinematics_parameters_file="$(arg kinematics_params)"
@@ -51,5 +53,7 @@
      use_fake_hardware="$(arg use_fake_hardware)"
      fake_sensor_commands="$(arg fake_sensor_commands)"
-     initial_positions="${initial_positions}" />
+     initial_positions="${initial_positions}" >
+       <origin xyz="0 0 ${robot_stand_height * 0.5}" rpy="0 0 2.355"/>
+    </xacro:ur_robot>
     <!-- instantiating robot arm and gripper -->
     <xacro:vacuum_gripper_definition prefix="${arm_prefix}" gripper_adjustment="0.01"/>
@@ -95,10 +99,4 @@
     </joint>
     <!-- end of arm-workcell link definitions -->
-    <!-- arm-workcell joint definitions -->
-    <joint name="stand_to_base" type="fixed">
-            <parent link="ur5_stand"/>
-            <child link="${arm_prefix}base_link"/>
-            <origin xyz="0 0 ${robot_stand_height * 0.5}" rpy="0 0 2.355"/>
-    </joint>
     <!-- end of arm workcell joint definitions-->
     <!-- arm-gripper coupling joint definitions -->

Commit message: cleaning up before PR

File: exercises/Perception-Driven_Manipulation/ros2/solution_ws/src/robot_workcell_support/urdf/ur5_workcell.xacro (robot description, xacro)
@@ -106,9 +106,4 @@
             <origin xyz="0 0 0" rpy="0 0 0"/> <!-- 0 1.57 0 -->
     </joint>
-    <!-- <joint name="world_frame_to_world" type="fixed">
-            <parent link="world"/>
-            <child link="world_frame"/>
-            <origin xyz="0 0 0" rpy="0 0 0"/>
-    </joint> -->
     <!-- end of arm-gripper coupling joint definitions -->
 </robot>

File: exercises/Perception-Driven_Manipulation/ros2/template_ws/src/robot_workcell_support/urdf/ur5_workcell.xacro (robot description, xacro)
@@ -106,9 +106,4 @@
             <origin xyz="0 0 0" rpy="0 0 0"/> <!-- 0 1.57 0 -->
     </joint>
-    <joint name="world_frame_to_world" type="fixed">
-            <parent link="world_frame"/>
-            <child link="world"/>
-            <origin xyz="0 0 0" rpy="0 0 0"/>
-    </joint>
     <!-- end of arm-gripper coupling joint definitions -->
 </robot>
